File: HSWR V2.kicad_pcb (KiCad board)
At the start: 4 copper layers, 152 x 139 mm, 161 parts, among them IC1 ADM3052, IC2 TPS65320C, IC4 INA240A1, IC5 INA240A1, P1 USB_B, P2 Interface, P3 IN+, P4 IN-, P5 MOTOR3, P6 MOTOR2, P7 MOTOR1, P8 SWD, Q1 ZXTC2045E6, Q10 ZXTC2045E6, Q11 IXFK230N20T, Q12 IXFK230N20T, Q2 ZXTC2045E6, Q3 IXFK230N20T, Q4 IXFK230N20T, Q5 ZXTC2045E6, Q6 ZXTC2045E6, Q7 IXFK230N20T, Q8 IXFK230N20T, Q9 ZXTC2045E6, U1 STM32F40X_LQFP64, U2 IR2110S, U3 IR2110S, U4 IR2110S, X1 8MHz 10ppm

Commit message: ~ removed/optionalised INA240 input filter ~ raised load resisitance of sense resistors for lower power loss ~ adopted old division factor on phase voltage sense deviders
Parts:
- C40, C42: value 220n -> opt
- Q11, Q12, Q3, Q4, Q7, Q8: value IXFK230N20T -> IRFP4668PBF
- R16, R17, R22, R23, R28, R29: value 4R7 -> 1R
- R49, R50, R51, R52: value 10R -> opt
- R53, R55, R57: value 64k9 -> 220k
- R54, R56, R58: value 1k -> k
- R7: value 64k9 -> 160k
- R8: value 1k -> 3k3
Connections:
- B1 pad 3: Net-(B1-Pad3) -> (no net)
- B1 pad 5: Net-(B1-Pad5) -> (no net)
- IC1 pad 10: Net-(IC1-Pad10) -> (no net)
- IC1 pad 4: /CAN bus transceiver/V+Sense -> (no net)
- P8 pad 6: Net-(P8-Pad6) -> (no net)
- U1 pad 11: Net-(U1-Pad11) -> (no net)
- U1 pad 2: Net-(U1-Pad2) -> (no net)
- U1 pad 28: Net-(U1-Pad28) -> (no net)
- U1 pad 3: Net-(U1-Pad3) -> (no net)
- U1 pad 33: /MCU/DC_CAL -> (no net)
- U1 pad 39: Net-(U1-Pad39) -> (no net)
- U1 pad 4: Net-(U1-Pad4) -> (no net)
- U1 pad 40: Net-(U1-Pad40) -> (no net)
- U1 pad 50: Net-(U1-Pad50) -> (no net)
- U1 pad 53: /MCU/FAULT -> (no net)
- U1 pad 54: Net-(U1-Pad54) -> (no net)
- U1 pad 55: Net-(U1-Pad55) -> (no net)
- U1 pad 56: Net-(U1-Pad56) -> (no net)
- U1 pad 9: Net-(U1-Pad9) -> (no net)

Commit message: - changed dividers to 220k vs 3k3 - changed hall supply to +5V instead of +3V3
Parts:
- R54, R56, R58: value k -> 3k3
- R7: value 160k -> 220k
Connections:
- P2 pad 7: +3V3 -> +5V
Routing:
- net +5V: track 62.1 -> 156.4 mm, vias 4 -> 6
Changed lines of the file:
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@@
-(kicad_pcb (version 4) (host pcbnew 4.0.1-stable)
+(kicad_pcb (version 4) (host pcbnew 4.0.7)
   (general
     (links 381)
-    (no_connects 2)
+    (no_connects 3)
     (area 66.949999 23.949999 219.050001 163.050001)
     (thickness 1.6)
     (drawings 14)
-    (tracks 1297)
+    (tracks 1307)
     (zones 0)
     (modules 161)
@@
       (effects (font (size 1 1) (thickness 0.15)))
     )
-    (fp_text value 160k (at 0 2.1 270) (layer F.Fab)
+    (fp_text value 220k (at 0 2.1 270) (layer F.Fab)
       (effects (font (size 1 1) (thickness 0.15)))
     )
@@
       (effects (font (size 1 1) (thickness 0.15)))
     )
-    (fp_text value k (at 0 2.1 90) (layer F.Fab)
+    (fp_text value 3k3 (at 0 2.1 90) (layer F.Fab)
       (effects (font (size 1 1) (thickness 0.15)))
     )
@@
       (effects (font (size 1 1) (thickness 0.15)))
     )
-    (fp_text value k (at 0 2.1 90) (layer F.Fab)
+    (fp_text value 3k3 (at 0 2.1 90) (layer F.Fab)
       (effects (font (size 1 1) (thickness 0.15)))
     )
@@
       (effects (font (size 1 1) (thickness 0.15)))
     )
-    (fp_text value k (at 0 2.1 90) (layer F.Fab)
+    (fp_text value 3k3 (at 0 2.1 90) (layer F.Fab)
       (effects (font (size 1 1) (thickness 0.15)))
     )
@@
       (net 2 Earth))
     (pad 7 thru_hole circle (at -3.81 1.27 90) (size 1.85 1.85) (drill 1.1) (layers *.Cu *.Mask F.SilkS)
-      (net 18 +3V3))
+      (net 37 +5V))
     (pad 8 thru_hole circle (at -3.81 -1.27 90) (size 1.85 1.85) (drill 1.1) (layers *.Cu *.Mask F.SilkS)
       (net 81 /Filters/HALL3_IN))
@@
   (segment (start 209.8 142.85) (end 209.8 143.6) (width 0.25) (layer F.Cu) (net 36))
   (segment (start 209.8 141.75) (end 209.8 142.85) (width 0.25) (layer F.Cu) (net 36))
+  (segment (start 166.39898 129) (end 163.14898 125.75) (width 0.25) (layer Power2) (net 37))
+  (segment (start 163.14898 125.75) (end 161.5 125.75) (width 0.25) (layer Power2) (net 37))
+  (segment (start 161.5 125.75) (end 104.25 125.75) (width 0.25) (layer Power2) (net 37))
+  (segment (start 102.5 125.75) (end 104.25 125.75) (width 0.25) (layer F.Cu) (net 37))
+  (via (at 104.25 125.75) (size 0.6) (drill 0.4) (layers F.Cu Power2) (net 37))
+  (segment (start 76.888147 126.5) (end 77.638147 125.75) (width 0.25) (layer Power2) (net 37))
+  (segment (start 77.638147 125.75) (end 102.5 125.75) (width 0.25) (layer Power2) (net 37))
+  (via (at 102.5 125.75) (size 0.6) (drill 0.4) (layers F.Cu Power2) (net 37))
+  (segment (start 74.27 127.81) (end 75.578147 127.81) (width 0.25) (layer Power2) (net 37))
+  (segment (start 75.578147 127.81) (end 76.888147 126.5) (width 0.25) (layer Power2) (net 37))
   (segment (start 166.39898 129) (end 184.7 129) (width 0.45) (layer Power2) (net 37))
   (segment (start 184.7 129) (end 187 131.3) (width 0.45) (layer Power2) (net 37))
