File: HSWR V2.kicad_pcb (KiCad board)
At the start: 4 copper layers, 152 x 139 mm, 161 parts, among them IC1 ADM3052, IC2 TPS65320C, IC4 INA240A1, IC5 INA240A1, P1 USB_B, P2 Interface, P3 IN+, P4 IN-, P5 MOTOR3, P6 MOTOR2, P7 MOTOR1, P8 SWD, Q1 ZXTC2045E6, Q10 ZXTC2045E6, Q11 IRFP4668PBF, Q12 IRFP4668PBF, Q2 ZXTC2045E6, Q3 IRFP4668PBF, Q4 IRFP4668PBF, Q5 ZXTC2045E6, Q6 ZXTC2045E6, Q7 IRFP4668PBF, Q8 IRFP4668PBF, Q9 ZXTC2045E6, U1 STM32F40X_LQFP64, U2 IR2110S, U3 IR2110S, U4 IR2110S, X1 8MHz 10ppm

Commit message: - updated project to 5.0.0 - added ignore file
Parts:
- removed REF** (x4): MountingHole_3.2mm_M3_Pad, Mounting_Holes:MountingHole_3.2mm_M3_Pad
- removed X1: 8MHz 10ppm, Crystals:Crystal_HC49-U_Vertical
- added Y1: 8MHz, Crystals:Crystal_HC49-U_Vertical, F.Cu at (153.0, 152.4)
Connections:
- B1 pad 3: (no net) -> Net-(B1-Pad3)
- B1 pad 5: (no net) -> Net-(B1-Pad5)
- C12 pad 2: GND -> Net-(C12-Pad2)
- C9 pad 2: Earth -> Net-(C9-Pad2)
- IC1 pad 10: (no net) -> Net-(IC1-Pad10)
- IC1 pad 16: Earth -> Net-(C9-Pad2)
- IC1 pad 2: GND -> Net-(C12-Pad2)
- IC1 pad 3: GND -> Net-(IC1-Pad3)
- IC1 pad 4: (no net) -> /CAN bus transceiver/V+Sense
- P8 pad 6: (no net) -> Net-(P8-Pad6)
- U1 pad 11: (no net) -> Net-(U1-Pad11)
- U1 pad 2: (no net) -> Net-(U1-Pad2)
- U1 pad 28: (no net) -> Net-(U1-Pad28)
- U1 pad 3: (no net) -> Net-(U1-Pad3)
- U1 pad 33: (no net) -> /MCU/DC_CAL
- U1 pad 39: (no net) -> Net-(U1-Pad39)
- U1 pad 4: (no net) -> Net-(U1-Pad4)
- U1 pad 40: (no net) -> Net-(U1-Pad40)
- U1 pad 50: (no net) -> Net-(U1-Pad50)
- U1 pad 53: (no net) -> /MCU/FAULT
- U1 pad 54: (no net) -> Net-(U1-Pad54)
- U1 pad 55: (no net) -> Net-(U1-Pad55)
- U1 pad 56: (no net) -> Net-(U1-Pad56)
- U1 pad 9: (no net) -> Net-(U1-Pad9)
Routing:
- net Net-(IC1-Pad3): vias 0 -> 1
- net Net-(C12-Pad2): vias 0 -> 1
- net GND: vias 50 -> 48

Commit message: - updated to VESC6 architecture - still some things to do in schematic
Parts:
- removed B1: MTC1, alexmod:MTC1
- removed C33, C34, C35, C36, C37, C38, C59, C60, C61: 100n, Capacitors_SMD:C_0805
- removed C39, C41: 10n, Capacitors_SMD:C_0805
- removed C40, C42: opt, Capacitors_SMD:C_0805
- removed C43, C44: 1u, Capacitors_SMD:C_0805
- removed C45: 10p, Capacitors_SMD:C_0805
- removed C46: 5n6, Capacitors_SMD:C_0805
- removed C47, C48: 10u, Capacitors_SMD:C_0805
- removed C49: 100u 6V3, Capacitors_ThroughHole:C_Radial_D6.3_L11.2_P2.5
- removed D7: RFN2L4S, Diodes_SMD:SMA_Standard
- removed D8, D9: D_Schottky, Diodes_SMD:SMA_Standard
- removed IC4, IC5: INA240A1, Housings_SSOP:TSSOP-8_4.4x3mm_Pitch0.65mm
- removed L1: SRR6038-3R3Y, alexmod:SRR6038
- removed P1: USB_B, alexmod:USBB_vert
- removed P2: Interface, alexmod:XG4A_20_wo_56
- removed P3: IN+, Mounting_Holes:MountingHole_6.5mm_Pad_Via
- removed P4: IN-, Mounting_Holes:MountingHole_6.5mm_Pad_Via
- removed P5: MOTOR3, Mounting_Holes:MountingHole_6.5mm_Pad_Via
- removed P6: MOTOR2, Mounting_Holes:MountingHole_6.5mm_Pad_Via
- removed P7: MOTOR1, Mounting_Holes:MountingHole_6.5mm_Pad_Via
- removed P8: SWD, Pin_Headers:Pin_Header_Straight_2x03
- removed Q1, Q10, Q2, Q5, Q6, Q9: ZXTC2045E6, TO_SOT_Packages_SMD:SOT-23-6
- removed R41: 30k1, Resistors_SMD:R_0805
- removed R42, R44: 95k3, Resistors_SMD:R_0805
- removed R43: 18k2, Resistors_SMD:R_0805
- removed R47, R48: CSS2H-3920R-L500, alexmod:CSS3920
- removed R49, R50, R51, R52: opt, Resistors_SMD:R_0805
- removed R53, R55, R57: 220k, Resistors_SMD:R_0805
- removed R54, R56, R58: 3k3, Resistors_SMD:R_0805
- added IC3: INA181, Package_TO_SOT_SMD:SOT-23-6, F.Cu at (-11.0, -7.17)
- added J10: SWD, Connector_PinHeader_2.54mm:PinHeader_2x03_P2.54mm_Vertical, F.Cu at (-64.2, 24.0)
- added J4: USB_B, Connector_USB:USB_B_TE_5787834_Vertical, F.Cu at (-57.0, -4.44)
- added J5: B+, MountingHole:MountingHole_6.5mm_Pad_Via, F.Cu at (-30.1, -2.22)
- added J6: B-, MountingHole:MountingHole_6.5mm_Pad_Via, F.Cu at (-45.7, 11.9)
- added J7: U, MountingHole:MountingHole_6.5mm_Pad_Via, F.Cu at (-59.2, 11.9)
- added J8: V, MountingHole:MountingHole_6.5mm_Pad_Via, F.Cu at (-43.7, -2.22)
- added J9: W, MountingHole:MountingHole_6.5mm_Pad_Via, F.Cu at (-32.1, 11.3)
- added JP1: 5V/3V3, Jumper:SolderJumper-3_P1.3mm_Open_RoundedPad1.0x1.5mm, F.Cu at (-21.0, -7.72)
- added JP2: opt., Jumper:SolderJumper-2_P1.3mm_Open_RoundedPad1.0x1.5mm, F.Cu at (-21.7, -4.89)
- added JP3: opt., Jumper:SolderJumper-2_P1.3mm_Open_RoundedPad1.0x1.5mm, F.Cu at (-18.3, -4.89)
- added NT1: Net-Tie_2, NetTie:NetTie-3_SMD_Pad0.5mm, F.Cu at (-45.7, 22.7)
- C1: value 100n -> 4n7; footprint Capacitors_SMD:C_0805 -> Capacitor_SMD:C_0805_2012Metric
- C10, C11, C12, C18, C19, C2, C20, C23, C24, C25, C32, C8, C9: footprint Capacitors_SMD:C_0805 -> Capacitor_SMD:C_0805_2012Metric
- C13, C14, C15, C16: value 4n7 -> 1u; footprint Capacitors_SMD:C_0805 -> Capacitor_SMD:C_0805_2012Metric
- C17, C22: value 15p -> 1u; footprint Capacitors_SMD:C_0805 -> Capacitor_SMD:C_0805_2012Metric
- C21: value 10n -> 1u; footprint Capacitors_SMD:C_0805 -> Capacitor_SMD:C_0805_2012Metric
- C26, C3, C4, C5: value 1u -> 4n7; footprint Capacitors_SMD:C_0805 -> Capacitor_SMD:C_0805_2012Metric
- C27, C28: value 22u -> 4n7; footprint Capacitors_SMD:C_1206 -> Capacitor_SMD:C_0805_2012Metric
- C29: value 100u 16V -> 4n7; footprint Capacitors_ThroughHole:C_Radial_D6.3_L11.2_P2.5 -> Capacitor_SMD:C_0805_2012Metric
- C30: value 10u -> 4n7; footprint Capacitors_SMD:C_0805 -> Capacitor_SMD:C_0805_2012Metric
- C31: value 3n3 -> 4n7; footprint Capacitors_SMD:C_0805 -> Capacitor_SMD:C_0805_2012Metric
- C50, C51, C53: footprint alexmod:C_Radial_D22_P10 -> Capacitor_THT:CP_Radial_D22.0mm_P10.00mm_SnapIn
- C52, C54, C55, C56, C57, C58: footprint Capacitors_SMD:C_2220 -> Capacitor_SMD:C_2220_5650Metric
- C6, C7: value 1u -> 15p; footprint Capacitors_SMD:C_0805 -> Capacitor_SMD:C_0805_2012Metric
- D1: value SS14 -> LED; footprint Diodes_SMD:SMA_Standard -> LED_SMD:LED_0805_2012Metric
- D2: footprint LEDs:LED_0805 -> LED_SMD:LED_0805_2012Metric
- D3: value GREEN -> LED; footprint LEDs:LED_0805 -> LED_SMD:LED_0805_2012Metric
- D4: value RED -> RFN2L4S; footprint LEDs:LED_0805 -> Diode_SMD:D_SMA
- D5, D6: footprint Diodes_SMD:SMA_Standard -> Diode_SMD:D_SMA
- IC1: value ADM3052 -> INA181; footprint Housings_SOIC:SOIC-16_7.5x10.3mm_Pitch1.27mm -> Package_TO_SOT_SMD:SOT-23-6
- IC2: value TPS65320C -> INA181; footprint alexmod:TSSOP-14_4.4x5mm_Pitch0.65mm_EP -> Package_TO_SOT_SMD:SOT-23-6
- Q11, Q12, Q3, Q4, Q7, Q8: value IRFP4668PBF -> IXFK300N20X3; footprint alexmod:TO-264_flat_reverse -> Package_TO_SOT_THT:TO-264-3_Horizontal_TabUp
- R1, R2: value 22R -> 1k; footprint Resistors_SMD:R_0805 -> Resistor_SMD:R_0805_2012Metric
- R10: value 10k -> NTC; footprint Resistors_SMD:R_0805 -> Resistor_SMD:R_0603_1608Metric
- R11: value R -> 10k; footprint Resistors_SMD:R_0805 -> Resistor_SMD:R_0805_2012Metric
- R12, R18, R19: value 120R -> 10k; footprint Resistors_SMD:R_0805 -> Resistor_SMD:R_0805_2012Metric
- R13: value 120R -> 2k2; footprint Resistors_SMD:R_0805 -> Resistor_SMD:R_0805_2012Metric
- R14, R15: value 10k -> 2k2; footprint Resistors_SMD:R_0805 -> Resistor_SMD:R_0805_2012Metric
- R16, R17, R20, R22, R23, R28, R29, R30, R6: footprint Resistors_SMD:R_0805 -> Resistor_SMD:R_0805_2012Metric
- R21: value 10k -> WSLF2512L5000FEB; footprint Resistors_SMD:R_0805 -> Resistor_SMD:R_2512_6332Metric
- R24, R25: value 120R -> WSLF2512L5000FEB; footprint Resistors_SMD:R_0805 -> Resistor_SMD:R_2512_6332Metric
- R26, R27, R32: value 10k -> 470R; footprint Resistors_SMD:R_0805 -> Resistor_SMD:R_0805_2012Metric
- R3, R4: value 2k2 -> 1k5; footprint Resistors_SMD:R_0805 -> Resistor_SMD:R_0805_2012Metric
- R31: footprint Resistors_SMD:R_1206 -> Resistor_SMD:R_0805_2012Metric
- R33, R34: value 2k2 -> 1k 0.1%; footprint Resistors_SMD:R_0805 -> Resistor_SMD:R_0805_2012Metric
- R35: value 2k2 -> 300k 0.1%; footprint Resistors_SMD:R_0805 -> Resistor_SMD:R_0805_2012Metric
- R36, R38: value 10k -> 4k7 0.1%; footprint Resistors_SMD:R_0805 -> Resistor_SMD:R_0805_2012Metric
- R37: value 10k -> 300k 0.1%; footprint Resistors_SMD:R_0805 -> Resistor_SMD:R_0805_2012Metric
- R39: value 52k3 -> 300k 0.1%; footprint Resistors_SMD:R_0805 -> Resistor_SMD:R_0805_2012Metric
- R40: value 28k -> 4k7 0.1%; footprint Resistors_SMD:R_0805 -> Resistor_SMD:R_0805_2012Metric
- R5: value 120R -> 470R; footprint Resistors_SMD:R_0805 -> Resistor_SMD:R_0805_2012Metric
- R7: value 220k -> 300k; footprint Resistors_SMD:R_0805 -> Resistor_SMD:R_0805_2012Metric
- R8: value 3k3 -> 4k7; footprint Resistors_SMD:R_0805 -> Resistor_SMD:R_0805_2012Metric
- R9: value NTC 10k -> 120R; footprint Resistors_SMD:R_0603 -> Resistor_SMD:R_0805_2012Metric
- U1: value STM32F40X_LQFP64 -> STM32F405RGTx; footprint Housings_QFP:LQFP-64_10x10mm_Pitch0.5mm -> Package_QFP:LQFP-64_10x10mm_P0.5mm
- U2, U3, U4: value IR2110S -> IRS2186; footprint Housings_SOIC:SOIC-16_7.5x10.3mm_Pitch1.27mm -> Package_SO:SO-8_3.9x4.9mm_P1.27mm
- Y1: footprint Crystals:Crystal_HC49-U_Vertical -> Crystal:Crystal_HC49-U_Vertical
Connections:
- net /MCU/DC_CAL renamed Net-(U1-Pad33)
- net /MCU/FAULT renamed Net-(U1-Pad53)
- C1 pad 1: GND -> /Filters/TEMP_IN
- C1 pad 2: /MCU/SERVO -> GND
- C13 pad 1: GND -> Net-(C13-Pad1)
- C13 pad 2: /Filters/TEMP_IN -> GND
- C14 pad 1: /Filters/HALL3_OUT -> +3V3
- C15 pad 1: /Filters/HALL2_OUT -> +3V3
- C16 pad 1: /Filters/HALL1_OUT -> +3V3
- C17 pad 1: Net-(C17-Pad1) -> +3V3
- C18 pad 1: Net-(C18-Pad1) -> +3V3
- C19 pad 1: Net-(C19-Pad1) -> +3V3
- C2 pad 1: /MCU/ADC_TEMP -> /MCU/TEMP_INT
- C20 pad 2: +3V3 -> +12V
- C21 pad 2: NRST -> +12V
- C22 pad 1: Net-(C22-Pad1) -> GND
- C22 pad 2: GND -> +12V
- C23 pad 1: GND -> Net-(C23-Pad1)
- C23 pad 2: +3V3 -> /Power MOSFETS/U
- C24 pad 1: GND -> Net-(C24-Pad1)
- C24 pad 2: +3V3 -> /Power MOSFETS/V
- C25 pad 1: GND -> Net-(C25-Pad1)
- C25 pad 2: +3V3 -> /Power MOSFETS/W
- C27 pad 1: +12VA -> GND
- C27 pad 2: Earth -> +3V3
- C28 pad 1: +12V -> GND
- C28 pad 2: GND -> +3V3
- C29 pad 1: +12V -> /MCU/U_I
- C3 pad 1: /Mosfet driver/H1_HI -> /Filters/HALL3_OUT
- C3 pad 2: /Mosfet driver/H1_VS -> GND
- C30 pad 1: +12V -> /MCU/V_I
- C31 pad 1: Net-(C31-Pad1) -> /MCU/W_I
- C32 pad 1: Net-(C32-Pad1) -> GND
- C32 pad 2: Net-(C32-Pad2) -> U2_REF
- C4 pad 1: +12V -> /Filters/HALL2_OUT
- C4 pad 2: /Mosfet driver/H1_LOW -> GND
- C5 pad 1: /Mosfet driver/H2_HI -> /Filters/HALL1_OUT
- C5 pad 2: /Mosfet driver/H2_VS -> GND
- C50 pad 2: GNDPWR -> Net-(C50-Pad2)
- C51 pad 2: GNDPWR -> Net-(C50-Pad2)
- C52 pad 2: /Mosfet driver/H1_LOW -> /Mosfet driver/U_VS
- C53 pad 2: GNDPWR -> Net-(C50-Pad2)
- C54 pad 2: /Mosfet driver/H1_LOW -> /Mosfet driver/U_VS
- C55 pad 2: GNDPWR -> /Mosfet driver/V_VS
- C56 pad 2: GNDPWR -> /Mosfet driver/V_VS
- C57 pad 2: /Mosfet driver/H3_LOW -> /Mosfet driver/W_VS
- C58 pad 2: /Mosfet driver/H3_LOW -> /Mosfet driver/W_VS
- C6 pad 1: +12V -> GND
- C6 pad 2: GNDPWR -> Net-(C6-Pad2)
- C7 pad 1: /Mosfet driver/H3_HI -> Net-(C7-Pad1)
- C7 pad 2: /Mosfet driver/H3_VS -> GND
- C8 pad 1: +12V -> Net-(C8-Pad1)
- C8 pad 2: /Mosfet driver/H3_LOW -> GND
- D1 pad 1: +5V -> GND
- D2 pad 1: Net-(D2-Pad1) -> GND
- D2 pad 2: GND -> Net-(D2-Pad2)
- D3 pad 1: Net-(D3-Pad1) -> GND
- D3 pad 2: GND -> Net-(D3-Pad2)
- D4 pad 1: Net-(D4-Pad1) -> Net-(C24-Pad1)
- D4 pad 2: GND -> +12V
- D5 pad 1: /Mosfet driver/H3_HI -> Net-(C25-Pad1)
- D6 pad 1: /Mosfet driver/H1_HI -> Net-(C23-Pad1)
- IC1 pad 1: (no net) -> Net-(IC1-Pad1)
- IC1 pad 2: Net-(C12-Pad2) -> GND
- IC1 pad 3: Net-(IC1-Pad3) -> /Mosfet driver/U_VS
- IC1 pad 4: /CAN bus transceiver/V+Sense -> GNDPWR
- IC1 pad 5: /CAN bus transceiver/CAN_RX -> U2_REF
- IC1 pad 6: /CAN bus transceiver/CAN_TX -> +3V3
- IC2 pad 1: Net-(C32-Pad1) -> Net-(IC2-Pad1)
- IC2 pad 2: +12V -> GND
- IC2 pad 3: +5V -> /Mosfet driver/V_VS
- IC2 pad 4: +3V3 -> GNDPWR
- IC2 pad 5: Net-(IC2-Pad5) -> U2_REF
- IC2 pad 6: Net-(D8-Pad1) -> +3V3
- Q11 pad 3: /Mosfet driver/H3_VS -> /Power MOSFETS/W
- Q12 pad 2: /Mosfet driver/H3_VS -> /Power MOSFETS/W
- Q12 pad 3: /Mosfet driver/H3_LOW -> /Mosfet driver/W_VS
- Q3 pad 3: /Mosfet driver/H1_VS -> /Power MOSFETS/U
- Q4 pad 2: /Mosfet driver/H1_VS -> /Power MOSFETS/U
- Q4 pad 3: /Mosfet driver/H1_LOW -> /Mosfet driver/U_VS
- Q7 pad 3: /Mosfet driver/H2_VS -> /Power MOSFETS/V
- Q8 pad 2: /Mosfet driver/H2_VS -> /Power MOSFETS/V
- Q8 pad 3: GNDPWR -> /Mosfet driver/V_VS
- R1 pad 1: /MCU/USB_DM -> /MCU/SCK_ADC_EXT
- R10 pad 1: /MCU/ADC_TEMP -> /MCU/TEMP_INT
- R10 pad 2: GND -> +3V3
- R11 pad 1: GNDPWR -> GND
- R11 pad 2: GND -> /MCU/TEMP_INT
- R12 pad 1: /Mosfet driver/M_H1 -> /Filters/TEMP_IN
- R12 pad 2: Net-(Q1-Pad4) -> +3V3
- R13 pad 1: /Mosfet driver/M_L1 -> /Filters/HALL3_IN
- R13 pad 2: Net-(Q2-Pad4) -> +3V3
- R14 pad 1: /Mosfet driver/H1_VS -> /Filters/HALL2_IN
- R14 pad 2: Net-(Q1-Pad4) -> +3V3
- R15 pad 1: /Mosfet driver/H1_LOW -> /Filters/HALL1_IN
- R15 pad 2: Net-(Q2-Pad4) -> +3V3
- R16 pad 2: Net-(Q1-Pad4) -> /Mosfet driver/U_GH
- R17 pad 2: Net-(Q2-Pad4) -> /Mosfet driver/U_GL
- R18 pad 1: /Mosfet driver/M_H2 -> /Filters/HALL3_IN
- R18 pad 2: Net-(Q5-Pad4) -> /Filters/HALL3_OUT
- R19 pad 1: /Mosfet driver/M_L2 -> /Filters/HALL2_IN
- R19 pad 2: Net-(Q6-Pad4) -> /Filters/HALL2_OUT
- R2 pad 1: /MCU/USB_DP -> /MCU/MISO_ADC_EXT2
- R20 pad 1: /Mosfet driver/H2_VS -> /Filters/HALL1_IN
- R20 pad 2: Net-(Q5-Pad4) -> /Filters/HALL1_OUT
- R21 pad 2: Net-(Q6-Pad4) -> /Mosfet driver/U_VS
- R22 pad 2: Net-(Q5-Pad4) -> /Mosfet driver/V_GH
- R23 pad 2: Net-(Q6-Pad4) -> /Mosfet driver/V_GL
- R24 pad 1: /Mosfet driver/M_H3 -> GNDPWR
- R24 pad 2: Net-(Q9-Pad4) -> /Mosfet driver/V_VS
- R25 pad 1: /Mosfet driver/M_L3 -> GNDPWR
- R25 pad 2: Net-(Q10-Pad4) -> /Mosfet driver/W_VS
- R26 pad 1: /Mosfet driver/H3_VS -> /MCU/U_I
- R26 pad 2: Net-(Q9-Pad4) -> Net-(IC1-Pad1)
- R27 pad 1: /Mosfet driver/H3_LOW -> /MCU/V_I
- R27 pad 2: Net-(Q10-Pad4) -> Net-(IC2-Pad1)
- R28 pad 2: Net-(Q9-Pad4) -> /Mosfet driver/W_GH
- R29 pad 2: Net-(Q10-Pad4) -> /Mosfet driver/W_GL
- R3 pad 1: Net-(P2-Pad19) -> GND
- R3 pad 2: /MCU/SERVO -> /MCU/SCK_ADC_EXT
- R32 pad 1: /Filters/TEMP_IN -> /MCU/W_I
- R32 pad 2: +3V3 -> Net-(IC3-Pad1)
- R33 pad 1: /Filters/HALL3_IN -> +3V3
- R33 pad 2: +3V3 -> U2_REF
- R34 pad 1: /Filters/HALL2_IN -> U2_REF
- R34 pad 2: +3V3 -> GND
- R35 pad 1: /Filters/HALL1_IN -> /Power MOSFETS/U
- R35 pad 2: +3V3 -> /MCU/U_U
- R36 pad 1: /Filters/HALL3_IN -> /MCU/U_U
- R36 pad 2: /Filters/HALL3_OUT -> GND
- R37 pad 1: /Filters/HALL2_IN -> /Power MOSFETS/V
- R37 pad 2: /Filters/HALL2_OUT -> /MCU/V_U
- R38 pad 1: /Filters/HALL1_IN -> /MCU/V_U
- R38 pad 2: /Filters/HALL1_OUT -> GND
- R39 pad 1: Net-(IC2-Pad9) -> /Power MOSFETS/W
- R39 pad 2: GND -> /MCU/W_U
- R4 pad 1: Net-(D2-Pad1) -> GND
- R4 pad 2: +3V3 -> /MCU/MISO_ADC_EXT2
- R40 pad 1: Net-(C46-Pad2) -> /MCU/W_U
- R40 pad 2: Net-(C45-Pad2) -> GND
- R5 pad 1: Net-(D3-Pad1) -> Net-(D1-Pad2)
- R5 pad 2: /MCU/LED_GREEN -> +3V3
- R6 pad 1: Net-(D4-Pad1) -> Net-(D2-Pad2)
- R6 pad 2: /MCU/LED_RED -> /MCU/LED_GREEN
- R7 pad 2: /MCU/AN_IN -> /MCU/BUS_U
- R8 pad 1: /MCU/AN_IN -> /MCU/BUS_U
- R9 pad 1: +3V3 -> Net-(D3-Pad2)
- R9 pad 2: /MCU/ADC_TEMP -> /MCU/LED_RED
- U1 pad 10: /MCU/AN_IN -> /MCU/W_I
- U1 pad 11: Net-(U1-Pad11) -> /MCU/BUS_U
- U1 pad 14: /MCU/SENS3 -> /MCU/U_U
- U1 pad 15: /MCU/SENS2 -> /MCU/V_U
- U1 pad 16: /MCU/SENS1 -> /MCU/W_U
- U1 pad 17: /MCU/ADC_TEMP -> /MCU/TEMP_INT
- U1 pad 20: /MCU/TX_SDA_NSS -> /MCU/RX_SDA_NSS
- U1 pad 23: /MCU/RX_SCL_MOSI -> /MCU/TX_SCL_MOSI
- U1 pad 24: /MCU/LED_GREEN -> /Filters/TEMP_IN
- U1 pad 25: /MCU/LED_RED -> Net-(U1-Pad25)
- U1 pad 26: /MCU/BR_SO2 -> /MCU/LED_GREEN
- U1 pad 27: /MCU/BR_SO1 -> /MCU/LED_RED
- U1 pad 29: /MCU/RX_SCL_MOSI -> /MCU/TX_SCL_MOSI
- U1 pad 30: /MCU/TX_SDA_NSS -> /MCU/RX_SDA_NSS
- U1 pad 31: Net-(C18-Pad1) -> Net-(C8-Pad1)
- U1 pad 34: /MCU/L3 -> /MCU/U_PWM_L
- U1 pad 35: /MCU/L2 -> /MCU/V_PWM_L
- U1 pad 36: /MCU/L1 -> /MCU/W_PWM_L
- U1 pad 37: /MCU/TX_SDA_NSS -> /Filters/HALL3_OUT
- U1 pad 38: /MCU/RX_SCL_MOSI -> /Filters/HALL2_OUT
- U1 pad 39: Net-(U1-Pad39) -> /Filters/HALL1_OUT
- U1 pad 41: /MCU/H3 -> /MCU/U_PWM_H
- U1 pad 42: /MCU/H2 -> /MCU/V_PWM_H
- U1 pad 43: /MCU/H1 -> /MCU/W_PWM_H
- U1 pad 47: Net-(C19-Pad1) -> Net-(C13-Pad1)
- U1 pad 5: Net-(C17-Pad1) -> Net-(C7-Pad1)
- U1 pad 51: /MCU/EN_GATE -> Net-(U1-Pad51)
- U1 pad 52: /Filters/HALL3_OUT -> Net-(U1-Pad52)
- U1 pad 57: /MCU/SERVO -> Net-(U1-Pad57)
- U1 pad 58: /Filters/HALL1_OUT -> /MCU/SERVO
- U1 pad 59: /Filters/HALL2_OUT -> Net-(U1-Pad59)
- U1 pad 6: Net-(C22-Pad1) -> Net-(C6-Pad2)
- U1 pad 8: /Filters/TEMP_IN -> /MCU/U_I
- U1 pad 9: Net-(U1-Pad9) -> /MCU/V_I
- U2 pad 1: /Mosfet driver/M_L3 -> /MCU/U_PWM_H
- U2 pad 2: /Mosfet driver/H3_LOW -> /MCU/U_PWM_L
- U2 pad 3: +12V -> GND
- U2 pad 6: /Mosfet driver/H3_VS -> /Power MOSFETS/U
- U2 pad 7: /Mosfet driver/H3_HI -> /Mosfet driver/U_GH
- U2 pad 8: /Mosfet driver/M_H3 -> Net-(C23-Pad1)
- U3 pad 1: /Mosfet driver/M_L1 -> /MCU/V_PWM_H
- U3 pad 2: /Mosfet driver/H1_LOW -> /MCU/V_PWM_L
- U3 pad 3: +12V -> GND
- U3 pad 6: /Mosfet driver/H1_VS -> /Power MOSFETS/V
- U3 pad 7: /Mosfet driver/H1_HI -> /Mosfet driver/V_GH
- U3 pad 8: /Mosfet driver/M_H1 -> Net-(C24-Pad1)
- U4 pad 1: /Mosfet driver/M_L2 -> /MCU/W_PWM_H
- U4 pad 2: GNDPWR -> /MCU/W_PWM_L
- U4 pad 3: +12V -> GND
- U4 pad 6: /Mosfet driver/H2_VS -> /Power MOSFETS/W
- U4 pad 7: /Mosfet driver/H2_HI -> /Mosfet driver/W_GH
- U4 pad 8: /Mosfet driver/M_H2 -> Net-(C25-Pad1)
- Y1 pad 1: Net-(C17-Pad1) -> Net-(C6-Pad2)
- Y1 pad 2: Net-(C22-Pad1) -> Net-(C7-Pad1)
Routing:
- net /MCU/LED_RED: track 3.77 -> 92.3 mm, vias 0 -> 4
- net /MCU/BR_SO1: track 88.5 -> 0.00 mm, vias 4 -> 0
- net /Mosfet driver/M_H1: track 83.7 -> 0.00 mm
- net /Filters/TEMP_IN: track 116.3 -> 200.1 mm, vias 2 -> 3
- net /MCU/LED_GREEN: track 4.57 -> 88.0 mm, vias 0 -> 4
- net /MCU/BR_SO2: track 83.5 -> 0.00 mm, vias 4 -> 0
- net /MCU/W_U: track 0.00 -> 79.5 mm, vias 0 -> 5
- net /MCU/U_U: track 0.00 -> 75.5 mm, vias 0 -> 3
- net /MCU/SENS3: track 75.5 -> 0.00 mm, vias 2 -> 0
- net /MCU/SENS1: track 75.2 -> 0.00 mm, vias 4 -> 0
- net /Mosfet driver/M_L3: track 70.4 -> 0.00 mm
- net /MCU/W_PWM_H: track 0.00 -> 66.6 mm, vias 0 -> 2
- net /MCU/H1: track 66.6 -> 0.00 mm, vias 2 -> 0
- net Net-(P2-Pad19): track 65.2 -> 0.00 mm
- net /MCU/U_PWM_H: track 0.00 -> 63.5 mm
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
Commit message: - started layout - high current path finished - some work on gate drivers
Parts:
- removed C51, C53: 330u 250V, Capacitor_THT:CP_Radial_D22.0mm_P10.00mm_SnapIn
- added C33: 330u 250V, Capacitor_THT:CP_Radial_D22.0mm_P10.00mm_SnapIn, F.Cu at (131.5, 93.5)
- added C34: 330u 250V, Capacitor_THT:CP_Radial_D22.0mm_P10.00mm_SnapIn, F.Cu at (155.0, 93.5)
- added C35: 330u 250V, Capacitor_THT:CP_Radial_D22.0mm_P10.00mm_SnapIn, F.Cu at (84.5, 93.5)
- added C36: 330u 250V, Capacitor_THT:CP_Radial_D22.0mm_P10.00mm_SnapIn, F.Cu at (108.0, 93.5)
- added D10: FR6J-TP, Diode_SMD:D_SMC, F.Cu at (161.5, 37.5)
- added D11: FR6J-TP, Diode_SMD:D_SMC, F.Cu at (148.0, 37.5)
- added D12: FR6J-TP, Diode_SMD:D_SMC, F.Cu at (119.5, 37.5)
- added D7: FR6J-TP, Diode_SMD:D_SMC, F.Cu at (77.5, 37.5)
- added D8: FR6J-TP, Diode_SMD:D_SMC, F.Cu at (104.0, 37.5)
- added D9: FR6J-TP, Diode_SMD:D_SMC, F.Cu at (190.0, 37.5)
- C20, C23, C24, C25, C52, C54, C55, C56, C57, C58: moved to F.Cu
- D4, D5, D6: footprint Diode_SMD:D_SMA -> Diode_SMD:D_SOD-123
- R21, R24, R25: value WSLF2512L5000FEB -> EWSL3920FL500S9; footprint Resistor_SMD:R_2512_6332Metric -> Resistor_SMD:R_4020_10251Metric
- moved NT1 266.7 mm to (209.0, 102.0), turned to 90 degrees
- moved J6 266.7 mm to (209.0, 91.0)
- moved J5 248.1 mm to (209.0, 64.0)
- moved J7 239.2 mm to (179.0, 33.0)
- moved J8 183.1 mm to (136.0, 33.0)
- moved J9 127.0 mm to (93.0, 33.0)
- moved R20 95.0 mm to (40.8, 64.4)
- moved C5 95.0 mm to (43.6, 61.4)
- moved R10 95.0 mm to (50.0, 54.2)
- moved R18 95.0 mm to (46.4, 64.4)
- moved R9 95.0 mm to (47.2, 54.2)
- moved C6 82.8 mm to (42.5, 119.8)
- moved R19 82.8 mm to (39.7, 116.8)
- moved C4 80.8 mm to (237.6, 63.8)
- moved R13 80.8 mm to (234.8, 60.8)
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Connections:
- C50 pad 2: Net-(C50-Pad2) -> GNDPWR
- C52 pad 2: /Mosfet driver/U_VS -> GNDPWR
- C54 pad 2: /Mosfet driver/U_VS -> GNDPWR
- C55 pad 2: /Mosfet driver/V_VS -> GNDPWR
- C56 pad 2: /Mosfet driver/V_VS -> GNDPWR
- C57 pad 2: /Mosfet driver/W_VS -> GNDPWR
- C58 pad 2: /Mosfet driver/W_VS -> GNDPWR
Routing:
- net +12V: track 354.9 -> 22.9 mm, vias 4 -> 0
- net /Filters/TEMP_IN: track 200.1 -> 0.00 mm, vias 3 -> 0
- net +3V3: track 176.9 -> 0.00 mm, vias 14 -> 0
- net GND: track 160.5 -> 0.00 mm, vias 37 -> 0
- net +5V: track 156.4 -> 0.00 mm, vias 6 -> 0
- net /MCU/EN_GATE: track 141.6 -> 0.00 mm, vias 2 -> 0
- net /Mosfet driver/H1_VS: track 108.4 -> 0.00 mm, vias 1 -> 0
- net /Mosfet driver/H2_VS: track 106.8 -> 0.00 mm
- net /Mosfet driver/H3_VS: track 105.7 -> 0.00 mm
- net /MCU/RX_SCL_MOSI: track 103.1 -> 0.00 mm, vias 3 -> 0
- net /MCU/TX_SDA_NSS: track 99.3 -> 0.00 mm, vias 2 -> 0
- net /Power MOSFETS/V: track 0.00 -> 97.4 mm, vias 0 -> 1
- net /Power MOSFETS/W: track 1.91 -> 99.1 mm, vias 0 -> 1
- net /MCU/ADC_TEMP: track 95.7 -> 0.00 mm, vias 4 -> 0
- net /Filters/HALL2_OUT: track 94.7 -> 0.00 mm
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- added copper zone on F.Cu, net +BATT
- added copper zone on F.Cu, net /Mosfet driver/U_VS
- added copper zone on F.Cu, net /Mosfet driver/V_VS
- added copper zone on F.Cu, net /Mosfet driver/W_VS
- added copper zone on B.Cu, net /Power MOSFETS/U
- added copper zone on F.Cu, net /Power MOSFETS/U
- added copper zone on Power1, net /Power MOSFETS/U
- added copper zone on B.Cu, net /Power MOSFETS/V
- added copper zone on F.Cu, net /Power MOSFETS/V
- added copper zone on Power1, net /Power MOSFETS/V
- added copper zone on B.Cu, net /Power MOSFETS/W
- added copper zone on F.Cu, net /Power MOSFETS/W
- added copper zone on Power1, net /Power MOSFETS/W
- added copper zone on F.Cu, net GNDPWR
- removed copper zone on B.Cu, net /Mosfet driver/H1_LOW
- removed copper zone on Power1, net /Mosfet driver/H1_VS
- removed copper zone on Power1, net /Mosfet driver/H2_VS
- removed copper zone on B.Cu, net /Mosfet driver/H3_LOW
- removed copper zone on Power1, net /Mosfet driver/H3_VS
- removed copper zone on B.Cu, net GNDPWR
Other:
- net class Default: via_dia 0.6 -> 0.8
- rule pad_to_mask_clearance: 0.2 -> 0.1

Commit message: - gate drivers routed - CSAs routed - HV/PA nets routed
Parts:
- added C37: 100n, Capacitor_SMD:C_0805_2012Metric, F.Cu at (88.5, 50.0)
- added C38: 100n, Capacitor_SMD:C_0805_2012Metric, F.Cu at (130.8, 50.0)
- added R41: 22R, Resistor_SMD:R_0805_2012Metric, F.Cu at (163.8, 141.5)
- added R42: 22R, Resistor_SMD:R_0805_2012Metric, F.Cu at (163.8, 139.5)
- added REF**: MountingHole_3.2mm_M3, MountingHole:MountingHole_3.2mm_M3, F.Cu at (167.0, 117.0)
- added REF**: MountingHole_3.2mm_M3, MountingHole:MountingHole_3.2mm_M3, F.Cu at (119.0, 117.0)
- added REF**: MountingHole_3.2mm_M3, MountingHole:MountingHole_3.2mm_M3, F.Cu at (71.0, 159.0)
- added REF**: MountingHole_3.2mm_M3, MountingHole:MountingHole_3.2mm_M3, F.Cu at (215.0, 159.0)
- added REF**: MountingHole_3.2mm_M3, MountingHole:MountingHole_3.2mm_M3, F.Cu at (215.0, 28.0)
- added REF**: MountingHole_3.2mm_M3, MountingHole:MountingHole_3.2mm_M3, F.Cu at (71.0, 28.0)
- C18, C19: moved to F.Cu
- C26: value 4n7 -> 1u; moved to F.Cu
- C27, C28: value 4n7 -> 1u
- moved J4 266.3 mm to (158.8, 151.6)
- moved R26 131.4 mm to (165.5, 124.5), turned to 90 degrees
- moved C8 129.7 mm to (171.7, 131.0), turned to 90 degrees
- moved IC1 129.3 mm to (167.8, 50.0), turned to 270 degrees
- moved R27 118.2 mm to (163.5, 124.5)
- moved IC2 117.0 mm to (125.8, 50.0), turned to 270 degrees
- moved IC3 110.4 mm to (83.5, 50.0), turned to 270 degrees
- moved C15 104.1 mm to (184.1, 137.7), turned to 0 degrees
- moved C26 104.0 mm to (170.8, 50.0)
- moved R35 103.8 mm to (186.2, 124.5), turned to 270 degrees
- moved R37 103.5 mm to (184.0, 124.5)
- moved C27 103.4 mm to (128.8, 50.0), turned to 270 degrees
- moved R36 101.8 mm to (186.2, 128.0)
- moved R38 101.6 mm to (184.0, 128.0)
- moved C16 95.3 mm to (177.7, 131.0), turned to 90 degrees
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Connections:
- J4 pad 2: /MCU/USB_DM -> Net-(J4-Pad2)
- J4 pad 3: /MCU/USB_DP -> Net-(J4-Pad3)
Routing:
- net +3V3: track 0.00 -> 197.2 mm, vias 0 -> 12
- net GND: track 0.00 -> 194.3 mm, vias 0 -> 6
- net U2_REF: track 0.00 -> 170.7 mm, vias 0 -> 4
- net Net-(IC3-Pad1): track 0.00 -> 144.8 mm, vias 0 -> 2
- net Net-(IC2-Pad1): track 0.00 -> 113.2 mm, vias 0 -> 2
- net /Power MOSFETS/W: track 99.1 -> 201.0 mm, vias 1 -> 2
- net /Power MOSFETS/U: track 33.0 -> 123.0 mm, vias 0 -> 2
- net /MCU/W_PWM_H: track 0.00 -> 89.6 mm, vias 0 -> 2
- net /MCU/W_PWM_L: track 0.00 -> 86.8 mm, vias 0 -> 2
- net /MCU/V_PWM_H: track 0.00 -> 82.9 mm, vias 0 -> 2
- net Net-(IC1-Pad1): track 0.00 -> 79.3 mm, vias 0 -> 2
- net /MCU/V_PWM_L: track 0.00 -> 76.8 mm, vias 0 -> 2
- net /Mosfet driver/V_GL: track 1.92 -> 78.3 mm, vias 1 -> 2
- net /Mosfet driver/U_GH: track 0.00 -> 71.6 mm, vias 0 -> 2
- net /Mosfet driver/U_GL: track 0.00 -> 70.3 mm, vias 0 -> 2
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Other:
- board text added: "HSWR V3.0 200V 100A *20170301 Alexander Schröder"
- board text removed: "HSWR V2.0 200V 100A *20170301 Alexander Schröder"

Commit message: - layout pretty much finished except PSU and maaaaybe R2D - started work on R2D with AD2S1205
Parts:
- added C39: 100n, Capacitor_SMD:C_0805_2012Metric, F.Cu at (151.5, 150.5)
- added C40: 100n, Capacitor_SMD:C_0805_2012Metric, F.Cu at (166.2, 151.0)
- added IC4: ADUM3054, Package_SO:SOIC-16W_7.5x10.3mm_P1.27mm, F.Cu at (93.0, 154.0)
- added IC5: ADuM4160, Package_SO:SOIC-16W_7.5x10.3mm_P1.27mm, F.Cu at (158.5, 154.8)
- added J1: IO, Auktora:PinHeader_2x10_P2.54mm_Vertical, F.Cu at (74.3, 135.4)
- added R43: 22R, Resistor_SMD:R_0805_2012Metric, F.Cu at (166.8, 158.5)
- added U5: AP1117-50, Package_TO_SOT_SMD:SOT-223-3_TabPin2, F.Cu at (76.5, 151.0)
- C10: value 10u -> 100n
- C9: value 1u -> 100n
- NT1: footprint NetTie:NetTie-3_SMD_Pad0.5mm -> NetTie:NetTie-2_SMD_Pad2.0mm
- R10: moved to B.Cu
- R31: value 300R -> 22R
- moved J10 288.9 mm to (192.2, 157.0), turned to 180 degrees
- moved R15 171.2 mm to (82.5, 127.0), turned to 270 degrees
- moved R13 169.2 mm to (79.0, 127.0), turned to 270 degrees
- moved R12 166.9 mm to (84.2, 127.0)
- moved JP1 165.4 mm to (80.0, 123.2)
- moved R14 164.9 mm to (80.8, 127.0)
- moved R2 163.1 mm to (79.5, 115.8), turned to 180 degrees
- moved R1 163.0 mm to (79.5, 120.8), turned to 180 degrees
- moved JP2 159.8 mm to (79.5, 118.8)
- moved R9 158.4 mm to (174.5, 148.5), turned to 90 degrees
- moved C7 156.7 mm to (187.2, 142.0), turned to 90 degrees
- moved C4 155.9 mm to (95.0, 127.0), turned to 270 degrees
- moved R4 154.1 mm to (82.2, 114.8)
- moved JP3 153.8 mm to (79.5, 113.8)
- moved C3 153.4 mm to (96.8, 127.0), turned to 270 degrees
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Connections:
- net Net-(J4-Pad3) renamed /USB/Host_D+
- C10 pad 1: Earth -> GNDD
- C11 pad 1: +12VA -> /CAN bus transceiver/12V_ext
- C12 pad 2: Net-(C12-Pad2) -> GND
- C9 pad 2: Net-(C9-Pad2) -> Earth
- J4 pad 1: Net-(J4-Pad1) -> /USB/VBUS
- J4 pad 2: Net-(J4-Pad2) -> /USB/Host_D-
- J4 pad 4: GND -> GNDD
- J4 pad 5: GND -> GNDD
- R31 pad 1: Net-(C10-Pad2) -> Net-(IC5-Pad11)
- R31 pad 2: +12VA -> /USB/Host_D-
- R41 pad 2: /MCU/USB_DP -> Net-(IC5-Pad10)
- R42 pad 1: Net-(J4-Pad2) -> /USB/Device_D-
- R42 pad 2: /MCU/USB_DM -> Net-(IC5-Pad11)
- U1 pad 26: /MCU/LED_GREEN -> Net-(U1-Pad26)
- U1 pad 27: /MCU/LED_RED -> Net-(U1-Pad27)
- U1 pad 44: /MCU/USB_DM -> /USB/Device_D-
- U1 pad 45: /MCU/USB_DP -> /USB/Device_D+
- U1 pad 50: Net-(U1-Pad50) -> /MCU/CAN_VSS_SENSE
- U1 pad 51: Net-(U1-Pad51) -> /MCU/LED_GREEN
- U1 pad 52: Net-(U1-Pad52) -> /MCU/LED_RED
Routing:
- net /MCU/TEMP_INT: track 0.00 -> 137.5 mm, vias 0 -> 2
- net /MCU/SERVO: track 0.00 -> 122.3 mm, vias 0 -> 2
- net /Filters/TEMP_IN: track 0.00 -> 116.4 mm, vias 0 -> 4
- net /MCU/RX_SDA_NSS: track 0.00 -> 112.7 mm, vias 0 -> 2
- net /MCU/TX_SCL_MOSI: track 0.00 -> 110.9 mm, vias 0 -> 2
- net /MCU/MISO_ADC_EXT2: track 0.00 -> 106.7 mm, vias 0 -> 2
- net /MCU/SCK_ADC_EXT: track 0.00 -> 106.3 mm, vias 0 -> 2
- net +12V: track 25.7 -> 116.2 mm
- net /Filters/HALL1_OUT: track 0.00 -> 89.2 mm, vias 0 -> 2
- net /CAN bus transceiver/CAN_TX: track 0.00 -> 87.2 mm, vias 0 -> 2
- net /Filters/HALL3_OUT: track 0.00 -> 87.1 mm
- net /Filters/HALL2_OUT: track 0.00 -> 86.6 mm
- net /CAN bus transceiver/CAN_RX: track 0.00 -> 86.5 mm, vias 0 -> 2
- net /MCU/CAN_VSS_SENSE: track 0.00 -> 84.8 mm, vias 0 -> 2
- net Earth: track 0.00 -> 52.3 mm, vias 0 -> 2
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- added copper zone on B.Cu, net GND
- added copper zone on F.Cu, net GND
