File: HSWR V2.sch (KiCad schematic (older format))
At the start: 29 parts, among them J1 CAN, J2 Motor, J3 IO, J4 USB_B, J5 B+, J6 B-, J7 U, J8 V, J9 W

Commit message: - layout pretty much finished except PSU and maaaaybe R2D - started work on R2D with AD2S1205
Parts:
- removed J1: CAN, symbol Connector:Conn_01x04_Male
- removed J2: Motor, symbol Connector:Conn_01x06_Male
- removed J3: IO, symbol Connector:Conn_01x08_Male
- removed R41, R42: 22R, Resistor_SMD:R_0805_2012Metric, symbol Device:R
- added J1: IO, Auktora:PinHeader_2x10_P2.54mm_Vertical, symbol Connector:Conn_01x20_Male
Connections:
- net labels added: GNDD
- net labels removed: +12VA
- wire segments 76 -> 88
- no-connect marks 1 -> 0
Other:
- moved on the sheet: J4
Changed lines of the file:
@@
 $Descr A4 11693 8268
 encoding utf-8
-Sheet 1 7
+Sheet 1 9
 Title "HSWR V2.0 200V 50A"
 Date "2017-02-05"
@@
 	1    0    0    -1
 $EndComp
-$Sheet
-S 1700 3700 850  400
-U 5899E225
-F0 "CAN bus transceiver" 40
-F1 "CAN.sch" 40
-F2 "CAN_RX" O R 2550 3800 60
-F3 "CAN_TX" I R 2550 3900 60
-F4 "CANH" I L 1700 3800 60
-F5 "CANL" I L 1700 3900 60
-F6 "V+Sense" O R 2550 4000 60
-$EndSheet
-$Sheet
-S 1700 4250 850  550
-U 5899E226
-F0 "Filters" 60
-F1 "hall_filters.sch" 60
-F2 "HALL3_IN" I L 1700 4400 40
-F3 "HALL2_IN" I L 1700 4500 40
-F4 "HALL1_IN" I L 1700 4600 40
-F5 "TEMP_IN" I L 1700 4700 40
-F6 "HALL3_OUT" O R 2550 4400 40
-F7 "HALL2_OUT" O R 2550 4500 40
-F8 "HALL1_OUT" O R 2550 4600 40
-F9 "TEMP_OUT" O R 2550 4700 40
-$EndSheet
 $Comp
 L power:+3V3 #PWR018
@@
 $EndSheet
 $Comp
-L power:+12VA #PWR022
-U 1 1 5899E265
-P 1300 3700
-F 0 "#PWR022" H 1300 3550 50  0001 C CNN
-F 1 "+12VA" V 1300 3950 50  0000 C CNN
-F 2 "" H 1300 3700 60  0000 C CNN
-F 3 "" H 1300 3700 60  0000 C CNN
-	1    1300 3700
-	0    1    1    0
-$EndComp
-NoConn ~ 2550 4000
-$Comp
 L power:Earth #PWR023
 U 1 1 5899E266
@@
 L Connector:USB_B J4
 U 1 1 5C9E7F89
-P 1400 2950
-F 0 "J4" H 1455 3417 50  0000 C CNN
-F 1 "USB_B" H 1455 3326 50  0000 C CNN
-F 2 "Connector_USB:USB_B_TE_5787834_Vertical" H 1550 2900 50  0001 C CNN
-F 3 " ~" H 1550 2900 50  0001 C CNN
-	1    1400 2950
+P 1050 2950
+F 0 "J4" H 1105 3417 50  0000 C CNN
+F 1 "USB_B" H 1105 3326 50  0000 C CNN
+F 2 "Connector_USB:USB_B_TE_5787834_Vertical" H 1200 2900 50  0001 C CNN
+F 3 " ~" H 1200 2900 50  0001 C CNN
+	1    1050 2950
 	1    0    0    -1
 $EndComp
 $Comp
-L power:GND #PWR0108
-U 1 1 5C9E8766
-P 1400 3350
-F 0 "#PWR0108" H 1400 3100 50  0001 C CNN
-F 1 "GND" H 1450 3200 50  0000 C CNN
-F 2 "" H 1400 3350 50  0001 C CNN
-F 3 "" H 1400 3350 50  0001 C CNN
-	1    1400 3350
-	1    0    0    -1
-$EndComp
-$Comp
-L power:GND #PWR0109
-U 1 1 5C9E87A0
-P 1300 3350
-F 0 "#PWR0109" H 1300 3100 50  0001 C CNN
-F 1 "GND" H 1250 3200 50  0000 C CNN
-F 2 "" H 1300 3350 50  0001 C CNN
-F 3 "" H 1300 3350 50  0001 C CNN
-	1    1300 3350
-	1    0    0    -1
-$EndComp
-$Comp
-L Connector:Conn_01x04_Male J1
-U 1 1 5C9E8BA0
-P 1100 3900
-F 0 "J1" H 1206 4178 50  0000 C CNN
-F 1 "CAN" H 950 3900 50  0000 C CNN
-F 2 "" H 1100 3900 50  0001 C CNN
-F 3 "~" H 1100 3900 50  0001 C CNN
-	1    1100 3900
-	1    0    0    1
-$EndComp
-$Comp
-L Connector:Conn_01x06_Male J2
-U 1 1 5C9E94FB
-P 1100 4600
-F 0 "J2" H 1206 4978 50  0000 C CNN
-F 1 "Motor" H 950 4600 50  0000 C CNN
-F 2 "" H 1100 4600 50  0001 C CNN
-F 3 "~" H 1100 4600 50  0001 C CNN
-	1    1100 4600
-	1    0    0    1
-$EndComp
-$Comp
 L power:GND #PWR0110
 U 1 1 5C9E9711
@@
 F24 "BUS_U" I R 4300 3800 50
 F25 "TEMP_M" I L 2950 4700 50
-F26 "CAN_RX" I L 2950 3800 50
-F27 "CAN_TX" I L 2950 3900 50
-F28 "HALL_1" I L 2950 4400 50
-F29 "HALL_2" I L 2950 4500 50
-F30 "HALL_3" I L 2950 4600 50
+F26 "HALL_1" I L 2950 4400 50
+F27 "HALL_2" I L 2950 4500 50
+F28 "HALL_3" I L 2950 4600 50
+F29 "CAN_VSS_SENSE" I L 2950 4000 50
+F30 "CAN_RX" I L 2950 3800 50
+F31 "CAN_TX" O L 2950 3900 50
 $EndSheet
 $Comp
@@
 	0    -1   -1   0
 $EndComp
-$Comp
-L Connector:Conn_01x08_Male J3
-U 1 1 5CA471B6
-P 1100 5550
-F 0 "J3" H 1206 6028 50  0000 C CNN
-F 1 "IO" H 1000 5550 50  0000 C CNN
-F 2 "" H 1100 5550 50  0001 C CNN
-F 3 "~" H 1100 5550 50  0001 C CNN
-	1    1100 5550
-	1    0    0    1
-$EndComp
-Wire Wire Line
-	1900 5350 1300 5350
-Connection ~ 1900 5350
-Wire Wire Line
-	1300 5450 2950 5450
-$Comp
-L power:GND #PWR0115
-U 1 1 5C9B9418
-P 1300 5150
-F 0 "#PWR0115" H 1300 4900 50  0001 C CNN
-F 1 "GND" V 1305 5022 50  0000 R CNN
-F 2 "" H 1300 5150 50  0001 C CNN
-F 3 "" H 1300 5150 50  0001 C CNN
-	1    1300 5150
-	0    -1   -1   0
-$EndComp
-Wire Wire Line
-	1300 5250 1700 5250
 Wire Wire Line
-	1700 5250 1700 6150
+	1300 4900 1700 4900
 Wire Wire Line
-	1300 5550 2950 5550
-Wire Wire Line
-	1300 5650 1900 5650
+	1700 4900 1700 6150
 Connection ~ 1900 5650
 $Comp
 L power:GND #PWR0116
 U 1 1 5C9D3F1A
-P 1300 5850
-F 0 "#PWR0116" H 1300 5600 50  0001 C CNN
-F 1 "GND" H 1305 5677 50  0000 C CNN
-F 2 "" H 1300 5850 50  0001 C CNN
-F 3 "" H 1300 5850 50  0001 C CNN
-	1    1300 5850
+P 1300 5400
+F 0 "#PWR0116" H 1300 5150 50  0001 C CNN
+F 1 "GND" H 1305 5227 50  0000 C CNN
+F 2 "" H 1300 5400 50  0001 C CNN
+F 3 "" H 1300 5400 50  0001 C CNN
+	1    1300 5400
 	0    -1   -1   0
 $EndComp
-Wire Wire Line
-	1300 5750 2950 5750
 $Comp
-L Device:R R41
-U 1 1 5C9C4B7D
-P 2250 2950
-F 0 "R41" V 2330 2950 50  0000 C CNN
-F 1 "22R" V 2250 2950 50  0000 C CNN
-F 2 "Resistor_SMD:R_0805_2012Metric" V 2180 2950 30  0001 C CNN
-F 3 "" H 2250 2950 30  0000 C CNN
-	1    2250 2950
-	0    -1   -1   0
+L Connector:Conn_01x20_Male J1
+U 1 1 5C9CF05F
+P 1100 4600
+F 0 "J1" H 1206 5678 50  0000 C CNN
+F 1 "IO" H 950 4600 50  0000 C CNN
+F 2 "Auktora:PinHeader_2x10_P2.54mm_Vertical" H 1100 4600 50  0001 C CNN
+F 3 "~" H 1100 4600 50  0001 C CNN
+	1    1100 4600
+	1    0    0    -1
 $EndComp
+$Sheet
+S 1700 4250 850  550
+U 5899E226
+F0 "Filters" 60
+F1 "hall_filters.sch" 60
+F2 "HALL3_IN" I L 1700 4400 40
+F3 "HALL2_IN" I L 1700 4500 40
+F4 "HALL1_IN" I L 1700 4600 40
+F5 "TEMP_IN" I L 1700 4700 40
+F6 "HALL3_OUT" O R 2550 4400 40
+F7 "HALL2_OUT" O R 2550 4500 40
+F8 "HALL1_OUT" O R 2550 4600 40
+F9 "TEMP_OUT" O R 2550 4700 40
+$EndSheet
+Wire Wire Line
+	1900 5150 1900 5000
+Wire Wire Line
+	1900 5000 1300 5000
+Connection ~ 1900 5150
+Wire Wire Line
+	1800 5450 1800 5100
+Wire Wire Line
+	1800 5100 1300 5100
+Wire Wire Line
+	1800 5450 2950 5450
+Wire Wire Line
+	1600 5550 1600 5200
+Wire Wire Line
+	1600 5200 1300 5200
+Wire Wire Line
+	1600 5550 2950 5550
+Wire Wire Line
+	1500 5650 1500 5300
+Wire Wire Line
+	1500 5300 1300 5300
 Wire Wire Line
-	2100 2950 1700 2950
+	1500 5650 1900 5650
 Wire Wire Line
-	2400 2950 2950 2950
+	1400 5750 1400 5500
+Wire Wire Line
+	1400 5500 1300 5500
+Wire Wire Line
+	1400 5750 2950 5750
 $Comp
-L Device:R R42
-U 1 1 5C9D445C
-P 2250 3050
-F 0 "R42" V 2330 3050 50  0000 C CNN
-F 1 "22R" V 2250 3050 50  0000 C CNN
-F 2 "Resistor_SMD:R_0805_2012Metric" V 2180 3050 30  0001 C CNN
-F 3 "" H 2250 3050 30  0000 C CNN
-	1    2250 3050
-	0    -1   1    0
+L power:GND #PWR04
+U 1 1 5C9F51F2
+P 1300 5600
+F 0 "#PWR04" H 1300 5350 50  0001 C CNN
+F 1 "GND" H 1305 5427 50  0000 C CNN
+F 2 "" H 1300 5600 50  0001 C CNN
+F 3 "" H 1300 5600 50  0001 C CNN
+	1    1300 5600
+	1    0    0    -1
 $EndComp
+$Sheet
+S 1700 3600 850  500
+U 5899E225
+F0 "CAN bus transceiver" 40
+F1 "CAN.sch" 40
+F2 "12V_ext" I L 1700 3700 50
+F3 "CAN_RX" O R 2550 3800 50
+F4 "CAN_TX" I R 2550 3900 50
+F5 "CANH" I L 1700 3800 50
+F6 "V+Sense" O R 2550 4000 50
+F7 "CANL" I L 1700 3900 50
+$EndSheet
+Wire Wire Line
+	1700 3700 1300 3700
+Wire Wire Line
+	2950 4000 2550 4000
+Wire Wire Line
+	2950 2950 2550 2950
+Wire Wire Line
+	2550 3050 2950 3050
 Wire Wire Line
-	2100 3050 1700 3050
+	1700 2950 1350 2950
 Wire Wire Line
-	2400 3050 2950 3050
+	1350 3050 1700 3050
+$Sheet
+S 1700 2600 850  700
+U 5CA14308
+F0 "USB" 50
+F1 "USB.sch" 50
+F2 "VBUS" I L 1700 2750 50
+F3 "Host_D-" B L 1700 3050 50
+F4 "Host_D+" B L 1700 2950 50
+F5 "Device_D-" B R 2550 3050 50
+F6 "Device_D+" B R 2550 2950 50
+$EndSheet
+Wire Wire Line
+	1350 2750 1700 2750
+$Comp
+L power:GNDD #PWR0108
+U 1 1 5CA2D976
+P 1050 3350
+F 0 "#PWR0108" H 1050 3100 50  0001 C CNN
+F 1 "GNDD" H 1054 3195 50  0000 C CNN
+F 2 "" H 1050 3350 50  0001 C CNN
+F 3 "" H 1050 3350 50  0001 C CNN
+	1    1050 3350
+	1    0    0    -1
+$EndComp
+$Comp
+L power:GNDD #PWR0109
+U 1 1 5CA2D9BA
+P 950 3350
+F 0 "#PWR0109" H 950 3100 50  0001 C CNN
+F 1 "GNDD" H 950 3100 50  0000 C CNN
+F 2 "" H 950 3350 50  0001 C CNN
+F 3 "" H 950 3350 50  0001 C CNN
+	1    950  3350
+	1    0    0    -1
+$EndComp
+$Sheet
+S 1700 1700 850  700
+U 5CA305B7
+F0 "R2D" 50
+F1 "R2D.sch" 50
+$EndSheet
 $EndSCHEMATC
