File: Power.sch (KiCad schematic (older format))
At the start: 35 parts, among them IC4 INA240A1, IC5 INA240A1, U2 IR2110S, U3 IR2110S, U4 IR2110S

Commit message: ~ removed/optionalised INA240 input filter ~ raised load resisitance of sense resistors for lower power loss ~ adopted old division factor on phase voltage sense deviders
Parts:
- C40, C42: value 220n -> opt
- R49, R50, R51, R52: value 10R -> opt
- R53, R55, R57: value 64k9 -> 220k
- R54, R56, R58: value 1k -> 12k
Changed lines of the file:
@@
 P 9900 1150
 F 0 "R53" V 9800 1150 50  0000 C CNN
-F 1 "64k9" V 9900 1150 50  0000 C CNN
+F 1 "220k" V 9900 1150 50  0000 C CNN
 F 2 "Resistors_SMD:R_0805" H 9900 1150 60  0001 C CNN
 F 3 "" H 9900 1150 60  0001 C CNN
@@
 P 9900 1250
 F 0 "R54" V 10000 1250 50  0000 C CNN
-F 1 "1k" V 9900 1250 50  0000 C CNN
+F 1 "12k" V 9900 1250 50  0000 C CNN
 F 2 "Resistors_SMD:R_0805" H 9900 1250 60  0001 C CNN
 F 3 "" H 9900 1250 60  0001 C CNN
@@
 P 9900 1750
 F 0 "R56" V 10000 1750 50  0000 C CNN
-F 1 "1k" V 9900 1750 50  0000 C CNN
+F 1 "12k" V 9900 1750 50  0000 C CNN
 F 2 "Resistors_SMD:R_0805" H 9900 1750 60  0001 C CNN
 F 3 "" H 9900 1750 60  0001 C CNN
@@
 P 9900 1650
 F 0 "R55" V 9800 1650 50  0000 C CNN
-F 1 "64k9" V 9900 1650 50  0000 C CNN
+F 1 "220k" V 9900 1650 50  0000 C CNN
 F 2 "Resistors_SMD:R_0805" H 9900 1650 60  0001 C CNN
 F 3 "" H 9900 1650 60  0001 C CNN
@@
 P 9900 2100
 F 0 "R57" V 9800 2100 50  0000 C CNN
-F 1 "64k9" V 9900 2100 50  0000 C CNN
+F 1 "220k" V 9900 2100 50  0000 C CNN
 F 2 "Resistors_SMD:R_0805" H 9900 2100 60  0001 C CNN
 F 3 "" H 9900 2100 60  0001 C CNN
@@
 P 9900 2200
 F 0 "R58" V 10000 2200 50  0000 C CNN
-F 1 "1k" V 9900 2200 50  0000 C CNN
+F 1 "12k" V 9900 2200 50  0000 C CNN
 F 2 "Resistors_SMD:R_0805" H 9900 2200 60  0001 C CNN
 F 3 "" H 9900 2200 60  0001 C CNN
@@
 P 4500 2400
 F 0 "R51" V 4580 2400 50  0000 C CNN
-F 1 "10R" V 4500 2400 50  0000 C CNN
+F 1 "opt" V 4500 2400 50  0000 C CNN
 F 2 "Resistors_SMD:R_0805" V 4430 2400 50  0001 C CNN
 F 3 "" H 4500 2400 50  0000 C CNN
@@
 P 4500 2700
 F 0 "R52" V 4580 2700 50  0000 C CNN
-F 1 "10R" V 4500 2700 50  0000 C CNN
+F 1 "opt" V 4500 2700 50  0000 C CNN
 F 2 "Resistors_SMD:R_0805" V 4430 2700 50  0001 C CNN
 F 3 "" H 4500 2700 50  0000 C CNN
@@
 P 4750 2550
 F 0 "C42" H 4775 2650 50  0000 L CNN
-F 1 "220n" H 4775 2450 50  0000 L CNN
+F 1 "opt" H 4775 2450 50  0000 L CNN
 F 2 "Capacitors_SMD:C_0805" H 4788 2400 50  0001 C CNN
 F 3 "" H 4750 2550 50  0000 C CNN
@@
 P 4450 6850
 F 0 "R49" V 4530 6850 50  0000 C CNN
-F 1 "10R" V 4450 6850 50  0000 C CNN
+F 1 "opt" V 4450 6850 50  0000 C CNN
 F 2 "Resistors_SMD:R_0805" V 4380 6850 50  0001 C CNN
 F 3 "" H 4450 6850 50  0000 C CNN
@@
 P 4450 7150
 F 0 "R50" V 4530 7150 50  0000 C CNN
-F 1 "10R" V 4450 7150 50  0000 C CNN
+F 1 "opt" V 4450 7150 50  0000 C CNN
 F 2 "Resistors_SMD:R_0805" V 4380 7150 50  0001 C CNN
 F 3 "" H 4450 7150 50  0000 C CNN
@@
 P 4700 7000
 F 0 "C40" H 4725 7100 50  0000 L CNN
-F 1 "220n" H 4725 6900 50  0000 L CNN
+F 1 "opt" H 4725 6900 50  0000 L CNN
 F 2 "Capacitors_SMD:C_0805" H 4738 6850 50  0001 C CNN
 F 3 "" H 4700 7000 50  0000 C CNN

Commit message: - changed dividers to 220k vs 3k3 - changed hall supply to +5V instead of +3V3
Parts:
- R54, R56, R58: value 12k -> 3k3
Changed lines of the file:
@@
 P 9900 1250
 F 0 "R54" V 10000 1250 50  0000 C CNN
-F 1 "12k" V 9900 1250 50  0000 C CNN
+F 1 "3k3" V 9900 1250 50  0000 C CNN
 F 2 "Resistors_SMD:R_0805" H 9900 1250 60  0001 C CNN
 F 3 "" H 9900 1250 60  0001 C CNN
@@
 P 9900 1750
 F 0 "R56" V 10000 1750 50  0000 C CNN
-F 1 "12k" V 9900 1750 50  0000 C CNN
+F 1 "3k3" V 9900 1750 50  0000 C CNN
 F 2 "Resistors_SMD:R_0805" H 9900 1750 60  0001 C CNN
 F 3 "" H 9900 1750 60  0001 C CNN
@@
 P 9900 2200
 F 0 "R58" V 10000 2200 50  0000 C CNN
-F 1 "12k" V 9900 2200 50  0000 C CNN
+F 1 "3k3" V 9900 2200 50  0000 C CNN
 F 2 "Resistors_SMD:R_0805" H 9900 2200 60  0001 C CNN
 F 3 "" H 9900 2200 60  0001 C CNN

Commit message: - updated project to 5.0.0 - added ignore file
Parts:
- C33, C34, C35, C36, C37, C38, C59, C60, C61: symbol C_Small -> Device:C_Small
- C39, C40, C41, C42, C43, C44: symbol C -> Device:C
- D5, D6, D7: symbol D_Small -> Device:D_Small
- IC4, IC5: symbol INA240 -> HSWR-V2-rescue:INA240
- R47, R48, R49, R50, R51, R52: symbol R -> Device:R
- R53, R54, R55, R56, R57, R58: symbol R-RESCUE-BLDC_4 -> HSWR-V2-rescue:R-RESCUE-BLDC_4
- U2, U3, U4: symbol IR2110S -> HSWR-V2-rescue:IR2110S
Connections:
- wire segments 79 -> 105

Commit message: - updated to VESC6 architecture - still some things to do in schematic
Parts:
- removed C33, C34, C35, C36, C37, C38, C59, C60, C61: 100n, Capacitors_SMD:C_0805, symbol Device:C_Small
- removed C39, C41: 10n, Capacitors_SMD:C_0805, symbol Device:C
- removed C40, C42: opt, Capacitors_SMD:C_0805, symbol Device:C
- removed C43, C44: 1u, Capacitors_SMD:C_0805, symbol Device:C
- removed D7: RFN2L4S, Diodes_SMD:SMA_Standard, symbol Device:D_Small
- removed IC4, IC5: INA240A1, Housings_SSOP:TSSOP-8_4.4x3mm_Pitch0.65mm, symbol HSWR-V2-rescue:INA240
- removed R47, R48: CSS2H-3920R-L500, alexmod:CSS3920, symbol Device:R
- removed R49, R50, R51, R52: opt, Resistors_SMD:R_0805, symbol Device:R
- removed R53, R55, R57: 220k, Resistors_SMD:R_0805, symbol HSWR-V2-rescue:R-RESCUE-BLDC_4
- removed R54, R56, R58: 3k3, Resistors_SMD:R_0805, symbol HSWR-V2-rescue:R-RESCUE-BLDC_4
- removed U2, U3, U4: IR2110S, Housings_SOIC:SOIC-16_7.5x10.3mm_Pitch1.27mm, symbol HSWR-V2-rescue:IR2110S
- added C20, C21, C22, C23, C24, C25: 1u, Capacitor_SMD:C_0805_2012Metric, symbol Device:C
- added C26, C27, C28, C29, C30, C31: 4n7, Capacitor_SMD:C_0805_2012Metric, symbol Device:C
- added C32: 100n, Capacitor_SMD:C_0805_2012Metric, symbol Device:C
- added D4: RFN2L4S, Diode_SMD:D_SMA, symbol Device:D_Small
- added IC1, IC2, IC3: INA181, Package_TO_SOT_SMD:SOT-23-6, symbol Auktoralib:INA181
- added R21, R24, R25: WSLF2512L5000FEB, Resistor_SMD:R_2512_6332Metric, symbol Device:R_Small
- added R26, R27, R32: 470R, Resistor_SMD:R_0805_2012Metric, symbol Device:R
- added R33, R34: 1k 0.1%, Resistor_SMD:R_0805_2012Metric, symbol Device:R
- added R35, R37, R39: 300k 0.1%, Resistor_SMD:R_0805_2012Metric, symbol Device:R
- added R36, R38, R40: 4k7 0.1%, Resistor_SMD:R_0805_2012Metric, symbol Device:R
- added U2, U3, U4: IRS2186, Package_SO:SO-8_3.9x4.9mm_P1.27mm, symbol Driver_FET:IRS2186
- D5, D6: footprint Diodes_SMD:SMA_Standard -> Diode_SMD:D_SMA
Connections:
- net labels added: U2_REF, U_GH, U_GL, U_I, U_PWM_H, U_PWM_L, U_U, U_VP, U_VS, V_GH, V_GL, V_I, V_PWM_H, V_PWM_L, V_U, V_VP, V_VS, W_GH, W_GL, W_I, W_PWM_H, W_PWM_L, W_U, W_VP, W_VS
- net labels removed: BR_SO1, BR_SO2, EN_GATE, H1, H1_HI, H1_LOW, H1_VL, H1_VS, H2, H2_HI, H2_LOW, H2_VL, H2_VS, H3, H3_HI, H3_LOW, H3_VL, H3_VS, L1, L2, L3, M_H1, M_H2, M_H3, M_L1, M_L2, M_L3, SENS1, SENS2, SENS3
- wire segments 105 -> 66
Other:
- moved on the sheet: D6

Commit message: - started layout - high current path finished - some work on gate drivers
Parts:
- D4, D5, D6: footprint Diode_SMD:D_SMA -> Diode_SMD:D_SOD-123
- R21, R24, R25: value WSLF2512L5000FEB -> EWSL3920FL500S9; footprint Resistor_SMD:R_2512_6332Metric -> Resistor_SMD:R_4020_10251Metric
Changed lines of the file:
@@
 F 0 "D6" H 3050 1780 50  0000 L CNN
 F 1 "RFN2L4S" H 2950 1620 50  0000 L CNN
-F 2 "Diode_SMD:D_SMA" V 3100 1700 50  0001 C CNN
+F 2 "Diode_SMD:D_SOD-123" V 3100 1700 50  0001 C CNN
 F 3 "" V 3100 1700 50  0000 C CNN
 	1    3100 1700
@@
 F 0 "D4" H 3050 3480 50  0000 L CNN
 F 1 "RFN2L4S" H 2950 3320 50  0000 L CNN
-F 2 "Diode_SMD:D_SMA" V 3100 3400 50  0001 C CNN
+F 2 "Diode_SMD:D_SOD-123" V 3100 3400 50  0001 C CNN
 F 3 "" V 3100 3400 50  0000 C CNN
 	1    3100 3400
@@
 F 0 "D5" H 3050 5230 50  0000 L CNN
 F 1 "RFN2L4S" H 2950 5070 50  0000 L CNN
-F 2 "Diode_SMD:D_SMA" V 3100 5150 50  0001 C CNN
+F 2 "Diode_SMD:D_SOD-123" V 3100 5150 50  0001 C CNN
 F 3 "" V 3100 5150 50  0000 C CNN
 	1    3100 5150
@@
 P 4550 2150
 F 0 "R21" H 4491 2104 50  0000 R CNN
-F 1 "WSLF2512L5000FEB" H 4491 2195 50  0000 R CNN
-F 2 "Resistor_SMD:R_2512_6332Metric" H 4550 2150 50  0001 C CNN
+F 1 "EWSL3920FL500S9" H 4491 2195 50  0000 R CNN
+F 2 "Resistor_SMD:R_4020_10251Metric" H 4550 2150 50  0001 C CNN
 F 3 "~" H 4550 2150 50  0001 C CNN
 	1    4550 2150
@@
 P 4550 3850
 F 0 "R24" H 4491 3804 50  0000 R CNN
-F 1 "WSLF2512L5000FEB" H 4491 3895 50  0000 R CNN
-F 2 "Resistor_SMD:R_2512_6332Metric" H 4550 3850 50  0001 C CNN
+F 1 "EWSL3920FL500S9" H 4491 3895 50  0000 R CNN
+F 2 "Resistor_SMD:R_4020_10251Metric" H 4550 3850 50  0001 C CNN
 F 3 "~" H 4550 3850 50  0001 C CNN
 	1    4550 3850
@@
 P 4550 5550
 F 0 "R25" H 4491 5504 50  0000 R CNN
-F 1 "WSLF2512L5000FEB" H 4491 5595 50  0000 R CNN
-F 2 "Resistor_SMD:R_2512_6332Metric" H 4550 5550 50  0001 C CNN
+F 1 "EWSL3920FL500S9" H 4491 5595 50  0000 R CNN
+F 2 "Resistor_SMD:R_4020_10251Metric" H 4550 5550 50  0001 C CNN
 F 3 "~" H 4550 5550 50  0001 C CNN
 	1    4550 5550

Commit message: - gate drivers routed - CSAs routed - HV/PA nets routed
Parts:
- added C37, C38: 100n, Capacitor_SMD:C_0805_2012Metric, symbol Device:C
- C26, C27, C28: value 4n7 -> 1u
- IC1, IC2, IC3: symbol Auktoralib:INA181 -> HSWR-V2-rescue:INA181-Auktoralib
- U2, U3, U4: symbol Driver_FET:IRS2186 -> HSWR-V2-rescue:IRS2186-Driver_FET
Connections:
- wire segments 66 -> 70
Changed lines of the file:
@@
 	9800 1150 9850 1150
 $Comp
-L Driver_FET:IRS2186 U2
+L HSWR-V2-rescue:IRS2186-Driver_FET U2
 U 1 1 5CA00151
 P 2450 2100
@@
 Connection ~ 2750 2200
 $Comp
-L Auktoralib:INA181 IC1
+L HSWR-V2-rescue:INA181-Auktoralib IC1
 U 1 1 5CA27007
 P 5100 2150
+AR Path="/5CA27007" Ref="IC1"  Part="1"
+AR Path="/5895E6A0/5CA27007" Ref="IC1"  Part="1"
 F 0 "IC1" H 5350 2500 50  0000 C CNN
 F 1 "INA181" H 5150 2200 50  0000 C CNN
@@
 P 5250 1500
 F 0 "C26" H 5135 1454 50  0000 R CNN
-F 1 "4n7" H 5135 1545 50  0000 R CNN
+F 1 "1u" H 5135 1545 50  0000 R CNN
 F 2 "Capacitor_SMD:C_0805_2012Metric" H 5288 1350 50  0001 C CNN
 F 3 "~" H 5250 1500 50  0001 C CNN
@@
 V_PWM_L
 $Comp
-L Driver_FET:IRS2186 U3
+L HSWR-V2-rescue:IRS2186-Driver_FET U3
 U 1 1 5CA74639
 P 2450 3800
@@
 Connection ~ 2750 3900
 $Comp
-L Auktoralib:INA181 IC2
+L HSWR-V2-rescue:INA181-Auktoralib IC2
 U 1 1 5CA7465B
 P 5100 3850
+AR Path="/5CA7465B" Ref="IC2"  Part="1"
+AR Path="/5895E6A0/5CA7465B" Ref="IC2"  Part="1"
 F 0 "IC2" H 5350 4200 50  0000 C CNN
 F 1 "INA181" H 5150 3900 50  0000 C CNN
@@
 	5950 3650 5900 3650
 Connection ~ 5900 3650
-Text GLabel 5600 3850 2    50   Input ~ 0
+Text GLabel 5950 3850 2    50   Input ~ 0
 U2_REF
 $Comp
@@
 P 5250 3200
 F 0 "C27" H 5135 3154 50  0000 R CNN
-F 1 "4n7" H 5135 3245 50  0000 R CNN
+F 1 "1u" H 5135 3245 50  0000 R CNN
 F 2 "Capacitor_SMD:C_0805_2012Metric" H 5288 3050 50  0001 C CNN
 F 3 "~" H 5250 3200 50  0001 C CNN
@@
 W_PWM_L
 $Comp
-L Driver_FET:IRS2186 U4
+L HSWR-V2-rescue:IRS2186-Driver_FET U4
 U 1 1 5CA75A04
 P 2450 5550
@@
 Connection ~ 2450 4800
 $Comp
-L Auktoralib:INA181 IC3
+L HSWR-V2-rescue:INA181-Auktoralib IC3
 U 1 1 5CA804F7
 P 5100 5550
+AR Path="/5CA804F7" Ref="IC3"  Part="1"
+AR Path="/5895E6A0/5CA804F7" Ref="IC3"  Part="1"
 F 0 "IC3" H 5350 5900 50  0000 C CNN
 F 1 "INA181" H 5150 5600 50  0000 C CNN
@@
 	5950 5350 5900 5350
 Connection ~ 5900 5350
-Text GLabel 5600 5550 2    50   Input ~ 0
+Text GLabel 5950 5550 2    50   Input ~ 0
 U2_REF
 $Comp
@@
 P 5250 4900
 F 0 "C28" H 5135 4854 50  0000 R CNN
-F 1 "4n7" H 5135 4945 50  0000 R CNN
+F 1 "1u" H 5135 4945 50  0000 R CNN
 F 2 "Capacitor_SMD:C_0805_2012Metric" H 5288 4750 50  0001 C CNN
 F 3 "~" H 5250 4900 50  0001 C CNN
@@
 	4700 5650 4550 5650
 Connection ~ 4550 5650
+$Comp
+L Device:C C37
+U 1 1 5C9BD3F3
+P 5900 4000
+F 0 "C37" H 5785 3954 50  0000 R CNN
+F 1 "100n" H 5785 4045 50  0000 R CNN
+F 2 "Capacitor_SMD:C_0805_2012Metric" H 5938 3850 50  0001 C CNN
+F 3 "~" H 5900 4000 50  0001 C CNN
+	1    5900 4000
+	-1   0    0    1
+$EndComp
+Wire Wire Line
+	5950 3850 5900 3850
+Connection ~ 5900 3850
+Wire Wire Line
+	5900 3850 5600 3850
+$Comp
+L power:GND #PWR01
+U 1 1 5C9BEC87
+P 5900 4150
+F 0 "#PWR01" H 5900 3900 50  0001 C CNN
+F 1 "GND" H 5905 3977 50  0000 C CNN
+F 2 "" H 5900 4150 50  0001 C CNN
+F 3 "" H 5900 4150 50  0001 C CNN
+	1    5900 4150
+	1    0    0    -1
+$EndComp
+$Comp
+L Device:C C38
+U 1 1 5C9BEF38
+P 5900 5700
+F 0 "C38" H 5785 5654 50  0000 R CNN
+F 1 "100n" H 5785 5745 50  0000 R CNN
+F 2 "Capacitor_SMD:C_0805_2012Metric" H 5938 5550 50  0001 C CNN
+F 3 "~" H 5900 5700 50  0001 C CNN
+	1    5900 5700
+	-1   0    0    1
+$EndComp
+$Comp
+L power:GND #PWR02
+U 1 1 5C9BEF3E
+P 5900 5850
+F 0 "#PWR02" H 5900 5600 50  0001 C CNN
+F 1 "GND" H 5905 5677 50  0000 C CNN
+F 2 "" H 5900 5850 50  0001 C CNN
+F 3 "" H 5900 5850 50  0001 C CNN
+	1    5900 5850
+	1    0    0    -1
+$EndComp
+Wire Wire Line
+	5950 5550 5900 5550
+Connection ~ 5900 5550
+Wire Wire Line
+	5900 5550 5600 5550
 $EndSCHEMATC
