File: CPU.sch (KiCad schematic (older format))
At the start: 13 parts, among them P8 SWD, U1 STM32F40X_LQFP64, X1 8MHz 10ppm

Commit message: - updated project to 5.0.0 - added ignore file
Parts:
- removed X1: 8MHz 10ppm, Crystals:Crystal_HC49-U_Vertical, symbol CRYSTAL_SMD
- added Y1: 8MHz, Crystals:Crystal_HC49-U_Vertical, symbol Device:Crystal
- C17, C18, C19, C20, C21, C22, C23, C24, C25, C26: symbol C-RESCUE-BLDC_4 -> HSWR-V2-rescue:C-RESCUE-BLDC_4
- P8: symbol CONN_6 -> HSWR-V2-rescue:CONN_6
- U1: symbol STM32F40X_LQFP64 -> HSWR-V2-rescue:STM32F40X_LQFP64
Connections:
- wire segments 53 -> 69
Changed lines of the file:
@@
-EESchema Schematic File Version 2
-LIBS:HSWR V2-rescue
-LIBS:power
-LIBS:device
-LIBS:transistors
-LIBS:conn
-LIBS:linear
-LIBS:regul
-LIBS:74xx
-LIBS:cmos4000
-LIBS:adc-dac
-LIBS:memory
-LIBS:xilinx
-LIBS:microcontrollers
-LIBS:dsp
-LIBS:microchip
-LIBS:analog_switches
-LIBS:motorola
-LIBS:texas
-LIBS:intel
-LIBS:audio
-LIBS:interface
-LIBS:digital-audio
-LIBS:philips
-LIBS:display
-LIBS:cypress
-LIBS:siliconi
-LIBS:opto
-LIBS:atmel
-LIBS:contrib
-LIBS:valves
+EESchema Schematic File Version 4
 LIBS:HSWR V2-cache
-EELAYER 25 0
+EELAYER 26 0
 EELAYER END
 $Descr A4 11693 8268
@@
 $EndDescr
 $Comp
-L STM32F40X_LQFP64 U1
+L HSWR-V2-rescue:STM32F40X_LQFP64 U1
 U 1 1 53F757A7
 P 5750 3900
@@
 $EndComp
 $Comp
-L C-RESCUE-BLDC_4 C19
+L HSWR-V2-rescue:C-RESCUE-BLDC_4 C19
 U 1 1 53F757AE
 P 7500 6350
@@
 $EndComp
 $Comp
-L C-RESCUE-BLDC_4 C18
+L HSWR-V2-rescue:C-RESCUE-BLDC_4 C18
 U 1 1 53F757B5
 P 7500 6100
@@
 $EndComp
 $Comp
-L GND-RESCUE-BLDC_4 #PWR039
+L HSWR-V2-rescue:GND-RESCUE-BLDC_4 #PWR039
 U 1 1 53F757BC
 P 7750 6400
@@
 $EndComp
 $Comp
-L GND-RESCUE-BLDC_4 #PWR040
+L HSWR-V2-rescue:GND-RESCUE-BLDC_4 #PWR040
 U 1 1 53F757C8
 P 7200 5150
@@
 $EndComp
 $Comp
-L C-RESCUE-BLDC_4 C17
+L HSWR-V2-rescue:C-RESCUE-BLDC_4 C17
 U 1 1 53F757DB
 P 7350 1800
@@
 $EndComp
 $Comp
-L C-RESCUE-BLDC_4 C22
+L HSWR-V2-rescue:C-RESCUE-BLDC_4 C22
 U 1 1 53F757E2
 P 8100 1800
@@
 $EndComp
 $Comp
-L GND-RESCUE-BLDC_4 #PWR041
+L HSWR-V2-rescue:GND-RESCUE-BLDC_4 #PWR041
 U 1 1 53F757E9
 P 8250 1600
@@
 $EndComp
 $Comp
-L GND-RESCUE-BLDC_4 #PWR042
+L HSWR-V2-rescue:GND-RESCUE-BLDC_4 #PWR042
 U 1 1 53F757EF
 P 7150 2550
@@
 SWCLK
 $Comp
-L C-RESCUE-BLDC_4 C20
+L HSWR-V2-rescue:C-RESCUE-BLDC_4 C20
 U 1 1 53F757F8
 P 7750 5450
@@
 NoConn ~ 4500 5450
 $Comp
-L GND-RESCUE-BLDC_4 #PWR043
+L HSWR-V2-rescue:GND-RESCUE-BLDC_4 #PWR043
 U 1 1 53F75856
 P 7950 3300
@@
 $EndComp
 Wire Wire Line
-	7950 3300 7950 3300
-Wire Wire Line
 	7200 5450 7200 5350
 Wire Wire Line
@@
 	7400 5650 7000 5650
 Wire Wire Line
-	7200 4200 7200 4650
+	7200 4200 7200 4350
 Wire Wire Line
 	7150 2350 7150 2550
@@
 	8100 1550 8100 1600
 Wire Wire Line
-	7350 1550 8250 1550
+	7350 1550 8100 1550
 Wire Wire Line
 	7350 1600 7350 1550
@@
 Connection ~ 8100 2050
 Wire Wire Line
-	7950 2050 8100 2050
+	7900 2050 8100 2050
 Wire Wire Line
-	8100 2000 8100 2250
+	8100 2000 8100 2050
 Wire Wire Line
 	7450 2250 7450 2150
@@
 	7450 2150 7000 2150
 Wire Wire Line
-	7000 2050 7550 2050
+	7000 2050 7350 2050
 Connection ~ 7200 4350
 Wire Wire Line
@@
 	7000 4950 7200 4950
 Wire Wire Line
-	7200 4950 7200 5150
+	7200 4950 7200 5050
 Wire Wire Line
-	7400 5100 7400 5650
+	7400 5100 7400 5150
 Connection ~ 7750 5750
 Wire Wire Line
@@
 Connection ~ 7750 6100
 Wire Wire Line
-	7750 5650 7750 6400
+	7750 5650 7750 5750
 Wire Wire Line
 	7750 6100 7700 6100
@@
 	7750 6350 7700 6350
 $Comp
-L C-RESCUE-BLDC_4 C21
+L HSWR-V2-rescue:C-RESCUE-BLDC_4 C21
 U 1 1 53F75896
 P 7950 3100
@@
 NoConn ~ 4500 4850
 $Comp
-L CONN_6 P8
+L HSWR-V2-rescue:CONN_6 P8
 U 1 1 53F77410
 P 10100 3150
@@
 $EndComp
 $Comp
-L GND-RESCUE-BLDC_4 #PWR044
+L HSWR-V2-rescue:GND-RESCUE-BLDC_4 #PWR044
 U 1 1 53F7741D
 P 9600 3100
@@
 NRST
 $Comp
-L C-RESCUE-BLDC_4 C23
+L HSWR-V2-rescue:C-RESCUE-BLDC_4 C23
 U 1 1 53F77426
 P 9400 1300
@@
 $EndComp
 $Comp
-L C-RESCUE-BLDC_4 C24
+L HSWR-V2-rescue:C-RESCUE-BLDC_4 C24
 U 1 1 53F7742D
 P 9650 1300
@@
 $EndComp
 $Comp
-L GND-RESCUE-BLDC_4 #PWR045
+L HSWR-V2-rescue:GND-RESCUE-BLDC_4 #PWR045
 U 1 1 53F7743B
 P 9100 1650
@@
 $EndComp
 $Comp
-L C-RESCUE-BLDC_4 C25
+L HSWR-V2-rescue:C-RESCUE-BLDC_4 C25
 U 1 1 53F77447
 P 9900 1300
@@
 $EndComp
 $Comp
-L C-RESCUE-BLDC_4 C26
+L HSWR-V2-rescue:C-RESCUE-BLDC_4 C26
 U 1 1 53F7744E
 P 10150 1300
@@
 $Bitmap
 Pos 1750 6700
-Scale 1,000000
+Scale 1.000000
 Data
 89 50 4E 47 0D 0A 1A 0A 00 00 00 0D 49 48 44 52 00 00 02 6A 00 00 02 41 08 02 00 00 00 79 DB 0E
@@
 $Bitmap
 Pos 3100 1050
-Scale 1,000000
+Scale 1.000000
 Data
 89 50 4E 47 0D 0A 1A 0A 00 00 00 0D 49 48 44 52 00 00 03 D4 00 00 00 CC 08 02 00 00 00 1D DB 7C
@@
 Text HLabel 4500 4950 0    60   Output ~ 0
 LED_GREEN
-$Comp
-L CRYSTAL_SMD X1
-U 1 1 540978A3
-P 7750 2050
-F 0 "X1" H 7750 2140 30  0000 C CNN
-F 1 "8MHz 10ppm" H 7800 1950 30  0000 L CNN
-F 2 "Crystals:Crystal_HC49-U_Vertical" H 7750 2050 60  0001 C CNN
-F 3 "" H 7750 2050 60  0000 C CNN
-F 4 "ABM3B-8.0-10-1UT" H 7750 2050 60  0001 C CNN "mfg#"
-	1    7750 2050
-	1    0    0    -1
-$EndComp
-$Comp
-L GND-RESCUE-BLDC_4 #PWR046
-U 1 1 54097D19
-P 7750 2150
-F 0 "#PWR046" H 7750 2150 30  0001 C CNN
-F 1 "GND" H 7750 2080 30  0001 C CNN
-F 2 "" H 7750 2150 60  0001 C CNN
-F 3 "" H 7750 2150 60  0001 C CNN
-	1    7750 2150
-	1    0    0    -1
-$EndComp
 Text HLabel 4500 2350 0    60   Input ~ 0
 MISO_ADC_EXT2
@@
 TX_SDA_NSS
 $Comp
-L +3V3 #PWR047
+L power:+3V3 #PWR047
 U 1 1 57529FFB
 P 7200 4200
@@
 $EndComp
 $Comp
-L +3V3 #PWR048
+L power:+3V3 #PWR048
 U 1 1 5752A2EE
 P 7400 5100
@@
 $EndComp
 $Comp
-L +3V3 #PWR049
+L power:+3V3 #PWR049
 U 1 1 5752A326
 P 7200 5350
@@
 $EndComp
 $Comp
-L +3V3 #PWR050
+L power:+3V3 #PWR050
 U 1 1 5752A907
 P 9750 2900
@@
 $EndComp
 $Comp
-L +3V3 #PWR051
+L power:+3V3 #PWR051
 U 1 1 5752A9C6
 P 9100 950
@@
 Connection ~ 7750 6350
 Wire Wire Line
-	9100 1000 10150 1000
+	9100 1000 9400 1000
+Wire Wire Line
+	9100 1600 9400 1600
+Wire Wire Line
+	7400 5150 7400 5650
+Wire Wire Line
+	8100 1550 8250 1550
+Wire Wire Line
+	7350 2050 7600 2050
+Wire Wire Line
+	8100 2050 8100 2250
+Wire Wire Line
+	7200 4350 7200 4450
+Wire Wire Line
+	7200 4450 7200 4550
 Wire Wire Line
-	9100 1600 10150 1600
+	7200 4550 7200 4650
+Wire Wire Line
+	7200 5050 7200 5150
+Wire Wire Line
+	7750 5750 7750 6100
+Wire Wire Line
+	7750 6100 7750 6350
+Wire Wire Line
+	9900 1600 10150 1600
+Wire Wire Line
+	9650 1600 9900 1600
+Wire Wire Line
+	9400 1600 9650 1600
+Wire Wire Line
+	9400 1000 9650 1000
+Wire Wire Line
+	9650 1000 9900 1000
+Wire Wire Line
+	9900 1000 10150 1000
+Wire Wire Line
+	7750 6350 7750 6400
+$Comp
+L Device:Crystal Y1
+U 1 1 5B6893E1
+P 7750 2050
+F 0 "Y1" H 7750 2318 50  0000 C CNN
+F 1 "8MHz" H 7750 2227 50  0000 C CNN
+F 2 "Crystals:Crystal_HC49-U_Vertical" H 7750 2050 50  0001 C CNN
+F 3 "~" H 7750 2050 50  0001 C CNN
+	1    7750 2050
+	1    0    0    -1
+$EndComp
 $EndSCHEMATC

Commit message: - updated to VESC6 architecture - still some things to do in schematic
Parts:
- removed C17, C22: 15p, Capacitors_SMD:C_0805, symbol HSWR-V2-rescue:C-RESCUE-BLDC_4
- removed C18, C19, C20, C23, C24, C25, C26: 1u, Capacitors_SMD:C_0805, symbol HSWR-V2-rescue:C-RESCUE-BLDC_4
- removed C21: 10n, Capacitors_SMD:C_0805, symbol HSWR-V2-rescue:C-RESCUE-BLDC_4
- removed P8: SWD, Pin_Headers:Pin_Header_Straight_2x03, symbol HSWR-V2-rescue:CONN_6
- removed U1: STM32F40X_LQFP64, Housings_QFP:LQFP-64_10x10mm_Pitch0.5mm, symbol HSWR-V2-rescue:STM32F40X_LQFP64
- added C13, C14, C15, C16, C17, C18, C19, C8: 1u, Capacitor_SMD:C_0805_2012Metric, symbol Device:C
- added C6, C7: 15p, Capacitor_SMD:C_0805_2012Metric, symbol Device:C
- added J10: SWD, Connector_PinHeader_2.54mm:PinHeader_2x03_P2.54mm_Vertical, symbol Connector:Conn_01x06_Male
- added U1: STM32F405RGTx, Package_QFP:LQFP-64_10x10mm_P0.5mm, symbol MCU_ST_STM32F4:STM32F405RGTx
- Y1: footprint Crystals:Crystal_HC49-U_Vertical -> Crystal:Crystal_HC49-U_Vertical
Connections:
- net labels added: BUS_U, RX_SDA_NSS, TEMP_INT, TEMP_M, TX_SCL_MOSI, U_I, U_PWM_H, U_PWM_L, U_U, V_I, V_PWM_H, V_PWM_L, V_U, W_I, W_PWM_H, W_PWM_L, W_U
- net labels removed: ADC_TEMP, AN_IN, BR_SO1, BR_SO2, DC_CAL, EN_GATE, FAULT, H1, H2, H3, L1, L2, L3, RX_SCL_MOSI, SENS1, SENS2, SENS3, TEMP_MOTOR, TX_SDA_NSS
- wire segments 69 -> 35
- no-connect marks 13 -> 16
Other:
- note removed: "Required for USB\nto work"

Commit message: - layout pretty much finished except PSU and maaaaybe R2D - started work on R2D with AD2S1205
Connections:
- net labels added: CAN_VSS_SENSE
- no-connect marks 16 -> 12
Changed lines of the file:
@@
 $Descr A4 11693 8268
 encoding utf-8
-Sheet 6 7
+Sheet 4 9
 Title "HSWR CPU"
 Date "2017-02-05"
@@
 	1    0    0    -1
 $EndComp
-$Comp
-L MCU_ST_STM32F4:STM32F405RGTx U1
-U 1 1 5C9EF5EF
-P 5700 3600
-F 0 "U1" H 5700 3500 50  0000 C CNN
-F 1 "STM32F405RGTx" H 5700 3600 50  0000 C CNN
-F 2 "Package_QFP:LQFP-64_10x10mm_P0.5mm" H 5100 1900 50  0001 R CNN
-F 3 "http://www.st.com/st-web-ui/static/active/en/resource/technical/document/datasheet/DM00037051.pdf" H 5700 3600 50  0001 C CNN
-	1    5700 3600
-	1    0    0    -1
-$EndComp
 Text HLabel 6400 2000 2    50   Input ~ 0
 U_U
@@
 Text HLabel 6400 3200 2    50   Input ~ 0
 USB_DP
-NoConn ~ 6400 3500
-Text HLabel 6400 3700 2    50   Input ~ 0
+Text HLabel 5000 4700 0    50   Input ~ 0
 LED_GREEN
-Text HLabel 6400 3800 2    50   Input ~ 0
+Text HLabel 5000 4800 0    50   Input ~ 0
 LED_RED
 Text HLabel 6400 4300 2    50   Input ~ 0
@@
 Text HLabel 6400 4500 2    50   Input ~ 0
 CAN_RX
-Text HLabel 6400 4600 2    50   Input ~ 0
+Text HLabel 6400 4600 2    50   Output ~ 0
 CAN_TX
 Text HLabel 6400 4700 2    50   Input ~ 0
@@
 NoConn ~ 6400 4100
 NoConn ~ 6400 4200
-NoConn ~ 6400 4400
 NoConn ~ 6400 4900
 Text HLabel 5000 3700 0    50   Input ~ 0
@@
 NoConn ~ 5000 4200
 NoConn ~ 5000 4600
-NoConn ~ 5000 4700
-NoConn ~ 5000 4800
 NoConn ~ 5000 4900
 NoConn ~ 5000 5000
@@
 	0    1    1    0
 $EndComp
+$Comp
+L MCU_ST_STM32F4:STM32F405RGTx U1
+U 1 1 5C9EF5EF
+P 5700 3600
+F 0 "U1" H 5700 3500 50  0000 C CNN
+F 1 "STM32F405RGTx" H 5700 3600 50  0000 C CNN
+F 2 "Package_QFP:LQFP-64_10x10mm_P0.5mm" H 5100 1900 50  0001 R CNN
+F 3 "http://www.st.com/st-web-ui/static/active/en/resource/technical/document/datasheet/DM00037051.pdf" H 5700 3600 50  0001 C CNN
+	1    5700 3600
+	1    0    0    -1
+$EndComp
+Text HLabel 6400 3500 2    50   Input ~ 0
+CAN_VSS_SENSE
 $EndSCHEMATC
