File: hall_filters.sch (KiCad schematic (older format))
At the start: 11 parts

Commit message: first commit of Amalga_100.
R2D needs to be finished.
Logicpart needs to be routed.
Parts:
- removed C1, C3, C4, C5: 4n7, Capacitor_SMD:C_0805_2012Metric, symbol Device:C
- removed R12, R18, R19, R20: 10k, Resistor_SMD:R_0805_2012Metric, symbol Device:R
- removed R13, R14, R15: 2k2, Resistor_SMD:R_0805_2012Metric, symbol Device:R
- added C13, C14, C15, C16: 4n7, Capacitor_SMD:C_0805_2012Metric, symbol Amalga_100-rescue:C-RESCUE-BLDC_4-HSWR-V2-rescue
- added R32, R36, R37, R38: 10k, Resistor_SMD:R_0805_2012Metric, symbol Amalga_100-rescue:R-RESCUE-BLDC_4-HSWR-V2-rescue
- added R33, R34, R35: 2k2, Resistor_SMD:R_0805_2012Metric, symbol Amalga_100-rescue:R-RESCUE-BLDC_4-HSWR-V2-rescue
Connections:
- wire segments 30 -> 31
