File: mosfets.sch (KiCad schematic (older format))
At the start: 29 parts, among them Q11 IXFK300N20X3, Q12 IXFK300N20X3, Q3 IXFK300N20X3, Q4 IXFK300N20X3, Q7 IXFK300N20X3, Q8 IXFK300N20X3

Commit message: - rescued schematic - added *.sch-bak to ignore - fixed bypass diode polarity - fixed PDEN being low - added 0R resistors instead of USB iso option - added caps to DCDC - added filter to VDDA
Parts:
- C33, C34, C35, C36, C50: symbol Device:CP -> HSWR-V2-rescue:CP-Device
- C52, C54, C55, C56, C57, C58: symbol Device:C -> HSWR-V2-rescue:C-Device
- D10, D11, D12, D7, D8, D9: symbol pspice:DIODE -> Device:D_Schottky
- Q11, Q12, Q3, Q4, Q7, Q8: symbol Device:Q_NMOS_GDS -> HSWR-V2-rescue:Q_NMOS_GDS-Device
- R16, R17, R22, R23, R28, R29: symbol Device:R -> HSWR-V2-rescue:R-Device
Connections:
- net +BATT: now also D11.1 (K), D8.1 (K), D9.1 (K); no longer D11.2 (A), D8.2 (A), D9.2 (A)
- net U: now also D10.1 (K), D9.2 (A); no longer D10.2 (A), D9.1 (K)
- net U_VS: now also D10.2 (A); no longer D10.1 (K)
- net V: now also D11.2 (A), D12.1 (K); no longer D11.1 (K), D12.2 (A)
- net V_VS: now also D12.2 (A); no longer D12.1 (K)
- net W: now also D7.1 (K), D8.2 (A); no longer D7.2 (A), D8.1 (K)
- net W_VS: now also D7.2 (A); no longer D7.1 (K)
Changed lines of the file:
@@
 EESchema Schematic File Version 4
-LIBS:HSWR V2-cache
-EELAYER 26 0
+EELAYER 30 0
 EELAYER END
 $Descr A4 11693 8268
@@
 Connection ~ 10050 3650
 $Comp
-L power:+BATT #PWR024
+L HSWR-V2-rescue:+BATT-power #PWR024
 U 1 1 575A4EA5
 P 10050 1700
@@
 $EndComp
 $Comp
-L Device:R R29
+L HSWR-V2-rescue:R-Device R29
 U 1 1 57621E05
 P 9550 4750
@@
 	10050 5400 10050 4950
 $Comp
-L Device:R R28
+L HSWR-V2-rescue:R-Device R28
 U 1 1 576296B6
 P 9550 2600
@@
 	9750 2600 9700 2600
 $Comp
-L Device:Q_NMOS_GDS Q12
+L HSWR-V2-rescue:Q_NMOS_GDS-Device Q12
 U 1 1 57637BFB
 P 9950 4750
@@
 $EndComp
 $Comp
-L Device:Q_NMOS_GDS Q11
+L HSWR-V2-rescue:Q_NMOS_GDS-Device Q11
 U 1 1 57637E5A
 P 9950 2600
@@
 Connection ~ 6600 3650
 $Comp
-L power:+BATT #PWR025
+L HSWR-V2-rescue:+BATT-power #PWR025
 U 1 1 589857E2
 P 6600 1700
@@
 $EndComp
 $Comp
-L Device:R R23
+L HSWR-V2-rescue:R-Device R23
 U 1 1 589857E8
 P 6100 4750
@@
 	6600 5400 6600 4950
 $Comp
-L Device:R R22
+L HSWR-V2-rescue:R-Device R22
 U 1 1 58985817
 P 6100 2600
@@
 	6300 2600 6250 2600
 $Comp
-L Device:Q_NMOS_GDS Q8
+L HSWR-V2-rescue:Q_NMOS_GDS-Device Q8
 U 1 1 5898584D
 P 6500 4750
@@
 $EndComp
 $Comp
-L Device:Q_NMOS_GDS Q7
+L HSWR-V2-rescue:Q_NMOS_GDS-Device Q7
 U 1 1 58985854
 P 6500 2600
@@
 Connection ~ 3150 3650
 $Comp
-L power:+BATT #PWR026
+L HSWR-V2-rescue:+BATT-power #PWR026
 U 1 1 58986AF5
 P 3150 1700
@@
 $EndComp
 $Comp
-L Device:R R17
+L HSWR-V2-rescue:R-Device R17
 U 1 1 58986AFB
 P 2700 4750
@@
 	3150 5400 3150 4950
 $Comp
-L Device:R R16
+L HSWR-V2-rescue:R-Device R16
 U 1 1 58986B2A
 P 2700 2600
@@
 $EndComp
 $Comp
-L Device:Q_NMOS_GDS Q4
+L HSWR-V2-rescue:Q_NMOS_GDS-Device Q4
 U 1 1 58986B60
 P 3050 4750
@@
 $EndComp
 $Comp
-L Device:Q_NMOS_GDS Q3
+L HSWR-V2-rescue:Q_NMOS_GDS-Device Q3
 U 1 1 58986B67
 P 3050 2600
@@
 	3150 1700 3150 2400
 $Comp
-L power:+BATT #PWR027
+L HSWR-V2-rescue:+BATT-power #PWR027
 U 1 1 58A716A6
 P 4250 7000
@@
 $EndComp
 $Comp
-L Device:C C52
+L HSWR-V2-rescue:C-Device C52
 U 1 1 58A7831F
 P 4550 7150
@@
 $EndComp
 $Comp
-L Device:C C54
+L HSWR-V2-rescue:C-Device C54
 U 1 1 58A78A84
 P 4800 7150
@@
 $EndComp
 $Comp
-L Device:C C55
+L HSWR-V2-rescue:C-Device C55
 U 1 1 58A797A9
 P 5050 7150
@@
 $EndComp
 $Comp
-L Device:C C56
+L HSWR-V2-rescue:C-Device C56
 U 1 1 58A797AF
 P 5300 7150
@@
 $EndComp
 $Comp
-L Device:C C57
+L HSWR-V2-rescue:C-Device C57
 U 1 1 58A799C2
 P 5550 7150
@@
 $EndComp
 $Comp
-L Device:C C58
+L HSWR-V2-rescue:C-Device C58
 U 1 1 58A799C8
 P 5800 7150
@@
 $EndComp
 $Comp
-L Device:CP C50
+L HSWR-V2-rescue:CP-Device C50
 U 1 1 58A7B8F0
 P 3200 7150
@@
 	3200 7300 3450 7300
 $Comp
-L Device:CP C34
+L HSWR-V2-rescue:CP-Device C34
 U 1 1 5C9BC25E
 P 3450 7150
@@
 Connection ~ 3450 7300
 $Comp
-L Device:CP C35
+L HSWR-V2-rescue:CP-Device C35
 U 1 1 5C9BC29A
 P 3700 7150
@@
 	3450 7300 3700 7300
 $Comp
-L Device:CP C36
+L HSWR-V2-rescue:CP-Device C36
 U 1 1 5C9BD172
 P 3950 7150
@@
 $EndComp
 $Comp
-L Device:CP C33
+L HSWR-V2-rescue:CP-Device C33
 U 1 1 5C9BD1B2
 P 2950 7150
@@
 	4250 7000 4550 7000
 $Comp
-L power:GNDPWR #PWR0166
+L HSWR-V2-rescue:GNDPWR-power #PWR0166
 U 1 1 5C9CC46D
 P 4250 7300
@@
 	4250 7300 3950 7300
 $Comp
-L pspice:DIODE D7
+L Device:D_Schottky D7
 U 1 1 5C9D0CA6
 P 10300 4750
+AR Path="/5C9D0CA6" Ref="D7"  Part="1"
+AR Path="/5895E67A/5C9D0CA6" Ref="D7"  Part="1"
 F 0 "D7" V 10346 4622 50  0000 R CNN
 F 1 "FR6J-TP" V 10255 4622 50  0000 R CNN
@@
 F 3 "" H 10300 4750 50  0001 C CNN
 	1    10300 4750
-	0    -1   -1   0
+	0    -1   1    0
 $EndComp
 Wire Wire Line
@@
 Connection ~ 10050 4950
 $Comp
-L pspice:DIODE D8
+L Device:D_Schottky D8
 U 1 1 5C9D9CB6
 P 10250 2600
+AR Path="/5C9D9CB6" Ref="D8"  Part="1"
+AR Path="/5895E67A/5C9D9CB6" Ref="D8"  Part="1"
 F 0 "D8" V 10296 2472 50  0000 R CNN
 F 1 "FR6J-TP" V 10205 2472 50  0000 R CNN
@@
 F 3 "" H 10250 2600 50  0001 C CNN
 	1    10250 2600
-	0    -1   -1   0
+	0    -1   1    0
 $EndComp
 Wire Wire Line
@@
 Connection ~ 10050 2400
 $Comp
-L pspice:DIODE D11
+L Device:D_Schottky D11
 U 1 1 5C9DC121
 P 6800 2600
+AR Path="/5C9DC121" Ref="D11"  Part="1"
+AR Path="/5895E67A/5C9DC121" Ref="D11"  Part="1"
 F 0 "D11" V 6846 2472 50  0000 R CNN
 F 1 "FR6J-TP" V 6755 2472 50  0000 R CNN
@@
 F 3 "" H 6800 2600 50  0001 C CNN
 	1    6800 2600
-	0    -1   -1   0
+	0    -1   1    0
 $EndComp
 Wire Wire Line
@@
 Connection ~ 6600 2800
 $Comp
-L pspice:DIODE D12
+L Device:D_Schottky D12
 U 1 1 5C9DE203
 P 6800 4750
+AR Path="/5C9DE203" Ref="D12"  Part="1"
+AR Path="/5895E67A/5C9DE203" Ref="D12"  Part="1"
 F 0 "D12" V 6846 4622 50  0000 R CNN
 F 1 "FR6J-TP" V 6755 4622 50  0000 R CNN
@@
 F 3 "" H 6800 4750 50  0001 C CNN
 	1    6800 4750
-	0    -1   -1   0
+	0    -1   1    0
 $EndComp
 Wire Wire Line
@@
 Connection ~ 6600 4950
 $Comp
-L pspice:DIODE D10
+L Device:D_Schottky D10
 U 1 1 5C9E04D1
 P 3350 4750
+AR Path="/5C9E04D1" Ref="D10"  Part="1"
+AR Path="/5895E67A/5C9E04D1" Ref="D10"  Part="1"
 F 0 "D10" V 3396 4622 50  0000 R CNN
 F 1 "FR6J-TP" V 3305 4622 50  0000 R CNN
@@
 F 3 "" H 3350 4750 50  0001 C CNN
 	1    3350 4750
-	0    -1   -1   0
+	0    -1   1    0
 $EndComp
 Wire Wire Line
@@
 Connection ~ 3150 4550
 $Comp
-L pspice:DIODE D9
+L Device:D_Schottky D9
 U 1 1 5C9E2B5A
 P 3350 2600
+AR Path="/5C9E2B5A" Ref="D9"  Part="1"
+AR Path="/5895E67A/5C9E2B5A" Ref="D9"  Part="1"
 F 0 "D9" V 3396 2472 50  0000 R CNN
 F 1 "FR6J-TP" V 3305 2472 50  0000 R CNN
@@
 F 3 "" H 3350 2600 50  0001 C CNN
 	1    3350 2600
-	0    -1   -1   0
+	0    -1   1    0
 $EndComp
 Wire Wire Line
@@
 	3350 2800 3150 2800
 Connection ~ 3150 2800
+Wire Wire Line
+	3350 2400 3350 2450
+Wire Wire Line
+	3350 2750 3350 2800
+Wire Wire Line
+	3350 4550 3350 4600
+Wire Wire Line
+	3350 4950 3350 4900
+Wire Wire Line
+	6800 4950 6800 4900
+Wire Wire Line
+	6800 4600 6800 4550
+Wire Wire Line
+	10300 4950 10300 4900
+Wire Wire Line
+	10300 4600 10300 4550
+Wire Wire Line
+	10250 2800 10250 2750
+Wire Wire Line
+	10250 2450 10250 2400
+Wire Wire Line
+	6800 2800 6800 2750
+Wire Wire Line
+	6800 2450 6800 2400
 $EndSCHEMATC
