File: mosfets.sch (KiCad schematic (older format))
At the start: 29 parts, among them Q11 IXFK300N20X3, Q12 IXFK300N20X3, Q3 IXFK300N20X3, Q4 IXFK300N20X3, Q7 IXFK300N20X3, Q8 IXFK300N20X3

Commit message: - changed CSA for Hall effect sensors - updated power stage layout
Parts:
- removed D10, D11, D12, D7, D8, D9: FR6J-TP, Diode_SMD:D_SMC, symbol Device:D_Schottky
- added C12, C26, C29: 100n, Capacitor_SMD:C_0805_2012Metric, symbol Device:C
- added C13, C27, C30: 1u, Capacitor_SMD:C_0805_2012Metric, symbol Device:C
- added C16, C28, C31: 4n7, Capacitor_SMD:C_0805_2012Metric, symbol Device:C
- added R20, R23, R26: 1k, Resistor_SMD:R_0805_2012Metric, symbol Device:R
- added U1, U2, U3: ACS781xLRTR-150B, Sensor_Current:Allegro_PSOF-7_4.8x6.4mm_P1.60mm, symbol Sensor_Current:ACS781xLRTR-150B
- C14: renamed from C33; symbol HSWR-V2-rescue:CP-Device -> Device:CP
- C15: renamed from C50; symbol HSWR-V2-rescue:CP-Device -> Device:CP
- C17: renamed from C34; symbol HSWR-V2-rescue:CP-Device -> Device:CP
- C18: renamed from C35; symbol HSWR-V2-rescue:CP-Device -> Device:CP
- C19: renamed from C36; symbol HSWR-V2-rescue:CP-Device -> Device:CP
- C20: renamed from C52; symbol HSWR-V2-rescue:C-Device -> Device:C
- C21: renamed from C54; symbol HSWR-V2-rescue:C-Device -> Device:C
- C22: renamed from C55; symbol HSWR-V2-rescue:C-Device -> Device:C
- C23: renamed from C56; symbol HSWR-V2-rescue:C-Device -> Device:C
- C24: renamed from C57; symbol HSWR-V2-rescue:C-Device -> Device:C
- C25: renamed from C58; symbol HSWR-V2-rescue:C-Device -> Device:C
- Q1: renamed from Q3; symbol HSWR-V2-rescue:Q_NMOS_GDS-Device -> Device:Q_NMOS_GDS
- Q2: renamed from Q4; symbol HSWR-V2-rescue:Q_NMOS_GDS-Device -> Device:Q_NMOS_GDS
- Q3: renamed from Q7; symbol HSWR-V2-rescue:Q_NMOS_GDS-Device -> Device:Q_NMOS_GDS
- Q4: renamed from Q8; symbol HSWR-V2-rescue:Q_NMOS_GDS-Device -> Device:Q_NMOS_GDS
- Q5: renamed from Q11; symbol HSWR-V2-rescue:Q_NMOS_GDS-Device -> Device:Q_NMOS_GDS
- Q6: renamed from Q12; symbol HSWR-V2-rescue:Q_NMOS_GDS-Device -> Device:Q_NMOS_GDS
- R18: renamed from R16; symbol HSWR-V2-rescue:R-Device -> Device:R
- R19: renamed from R17; symbol HSWR-V2-rescue:R-Device -> Device:R
- R21: renamed from R22; symbol HSWR-V2-rescue:R-Device -> Device:R
- R22: renamed from R23; symbol HSWR-V2-rescue:R-Device -> Device:R
- R24: renamed from R28; symbol HSWR-V2-rescue:R-Device -> Device:R
- R25: renamed from R29; symbol HSWR-V2-rescue:R-Device -> Device:R
Connections:
- net labels added: +3V3, GND, U_I, V_I, W_I
- wire segments 71 -> 53
- no-connect marks 0 -> 6
Other:
- moved on the sheet: R18, R19, R21, R22, R24, R25

Commit message: - fixed ISP connector being mirrored - changed some footprints to get them 3D Models - added a preliminary BOM
Parts:
- C24: footprint Capacitor_SMD:C_2220_5650Metric -> Crystal:Crystal_HC49-4H_Vertical
Changed lines of the file:
@@
 F 0 "C24" H 5500 6900 50  0000 L CNN
 F 1 "2u2 250V" V 5550 7400 50  0000 L CNN
-F 2 "Capacitor_SMD:C_2220_5650Metric" H 5588 7000 50  0001 C CNN
+F 2 "Crystal:Crystal_HC49-4H_Vertical" H 5588 7000 50  0001 C CNN
 F 3 "" H 5550 7150 50  0000 C CNN
 	1    5550 7150

Commit message: - removed some unused symbols from HSWR.lib - changed U8 (linear reg) to standard symbol - fixed wrong footprint for C24
Parts:
- C24: footprint Crystal:Crystal_HC49-4H_Vertical -> Capacitor_SMD:C_2220_5650Metric
Changed lines of the file:
@@
 F 0 "C24" H 5500 6900 50  0000 L CNN
 F 1 "2u2 250V" V 5550 7400 50  0000 L CNN
-F 2 "Crystal:Crystal_HC49-4H_Vertical" H 5588 7000 50  0001 C CNN
+F 2 "Capacitor_SMD:C_2220_5650Metric" H 5588 7000 50  0001 C CNN
 F 3 "" H 5550 7150 50  0000 C CNN
 	1    5550 7150
