File: CAN.sch (KiCad schematic (older format))
At the start: 6 parts, among them IC4 ADUM3054, U8 AP1117-50

Commit message: - renamed ADUM3054 as ADM3054 - specified ADuM120N1 (fail high)
Parts:
- IC4: value ADUM3054 -> ADM3054
Changed lines of the file:
@@
 AR Path="/5899E225/5CA06D6C" Ref="IC4"  Part="1"
 F 0 "IC4" H 5500 2850 50  0000 C CNN
-F 1 "ADUM3054" H 6350 3900 50  0000 C CNN
+F 1 "ADM3054" H 6350 3900 50  0000 C CNN
 F 2 "Package_SO:SOIC-16W_7.5x10.3mm_P1.27mm" H 5950 3300 50  0001 C CNN
 F 3 "" H 5950 3300 50  0001 C CNN
