File: CAN.kicad_sch (KiCad schematic)
At the start: 6 parts, among them IC4 ADM3054, U8 AP1117-50

Commit message: - some work on schematic
Parts:
- renumbered C52 to C5, C53 to C6, C54 to C7, IC4 to IC2, R40 to R15, U8 to U2
Changed lines of the file:
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@@
   (symbol (lib_id "Device:C_Small") (at 144.78 66.04 0) (mirror y) (unit 1)
     (in_bom yes) (on_board yes) (dnp no)
-    (property "Reference" "C53" (at 142.24 66.04 0)
+    (property "Reference" "C6" (at 142.24 66.04 0)
       (effects (font (size 1.27 1.27)) (justify left))
     )
@@
       (project "HSWR"
         (path "/51094070-255e-40e7-bed5-d199e288e5dd/00000000-0000-0000-0000-00005899e225"
-          (reference "C53") (unit 1)
+          (reference "C6") (unit 1)
         )
       )
@@
   (symbol (lib_id "Device:C_Small") (at 110.49 66.04 0) (mirror y) (unit 1)
     (in_bom yes) (on_board yes) (dnp no)
-    (property "Reference" "C52" (at 106.68 66.04 0)
+    (property "Reference" "C5" (at 106.68 66.04 0)
       (effects (font (size 1.27 1.27)) (justify left))
     )
@@
       (project "HSWR"
         (path "/51094070-255e-40e7-bed5-d199e288e5dd/00000000-0000-0000-0000-00005899e225"
-          (reference "C52") (unit 1)
+          (reference "C5") (unit 1)
         )
       )
@@
   (symbol (lib_id "power:Earth") (at 118.11 71.12 0) (mirror y) (unit 1)
     (in_bom yes) (on_board yes) (dnp no)
-    (property "Reference" "#PWR0102" (at 118.11 77.47 0)
+    (property "Reference" "#PWR027" (at 118.11 77.47 0)
       (effects (font (size 1.27 1.27)) hide)
     )
@@
       (project "HSWR"
         (path "/51094070-255e-40e7-bed5-d199e288e5dd/00000000-0000-0000-0000-00005899e225"
-          (reference "#PWR0102") (unit 1)
+          (reference "#PWR027") (unit 1)
         )
       )
@@
   (symbol (lib_id "power:GND") (at 153.67 102.87 0) (unit 1)
     (in_bom yes) (on_board yes) (dnp no)
-    (property "Reference" "#PWR0106" (at 153.67 109.22 0)
+    (property "Reference" "#PWR032" (at 153.67 109.22 0)
       (effects (font (size 1.27 1.27)) hide)
     )
@@
       (project "HSWR"
         (path "/51094070-255e-40e7-bed5-d199e288e5dd/00000000-0000-0000-0000-00005899e225"
-          (reference "#PWR0106") (unit 1)
+          (reference "#PWR032") (unit 1)
         )
       )
@@
   (symbol (lib_id "Device:R_Small") (at 135.89 82.55 0) (mirror y) (unit 1)
     (in_bom yes) (on_board yes) (dnp no)
-    (property "Reference" "R40" (at 138.43 83.82 90)
+    (property "Reference" "R15" (at 138.43 83.82 90)
       (effects (font (size 1.27 1.27)) (justify left))
     )
@@
       (project "HSWR"
         (path "/51094070-255e-40e7-bed5-d199e288e5dd/00000000-0000-0000-0000-00005899e225"
-          (reference "R40") (unit 1)
+          (reference "R15") (unit 1)
         )
       )
@@
   (symbol (lib_id "Device:C_Small") (at 157.48 66.04 0) (unit 1)
     (in_bom yes) (on_board yes) (dnp no)
-    (property "Reference" "C54" (at 161.29 66.04 0)
+    (property "Reference" "C7" (at 161.29 66.04 0)
       (effects (font (size 1.27 1.27)) (justify left))
     )
@@
       (project "HSWR"
         (path "/51094070-255e-40e7-bed5-d199e288e5dd/00000000-0000-0000-0000-00005899e225"
-          (reference "C54") (unit 1)
+          (reference "C7") (unit 1)
         )
       )
@@
   (symbol (lib_id "power:+3V3") (at 157.48 63.5 0) (unit 1)
     (in_bom yes) (on_board yes) (dnp no)
-    (property "Reference" "#PWR0108" (at 157.48 67.31 0)
+    (property "Reference" "#PWR034" (at 157.48 67.31 0)
       (effects (font (size 1.27 1.27)) hide)
     )
@@
       (project "HSWR"
         (path "/51094070-255e-40e7-bed5-d199e288e5dd/00000000-0000-0000-0000-00005899e225"
-          (reference "#PWR0108") (unit 1)
+          (reference "#PWR034") (unit 1)
         )
       )
@@
   (symbol (lib_id "power:+12VA") (at 110.49 63.5 0) (unit 1)
     (in_bom yes) (on_board yes) (dnp no)
-    (property "Reference" "#PWR0100" (at 110.49 67.31 0)
+    (property "Reference" "#PWR025" (at 110.49 67.31 0)
       (effects (font (size 1.27 1.27)) hide)
     )
@@
       (project "HSWR"
         (path "/51094070-255e-40e7-bed5-d199e288e5dd/00000000-0000-0000-0000-00005899e225"
-          (reference "#PWR0100") (unit 1)
+          (reference "#PWR025") (unit 1)
         )
       )
@@
   (symbol (lib_id "HSWR:ADUM3054") (at 151.13 86.36 0) (mirror y) (unit 1)
     (in_bom yes) (on_board yes) (dnp no)
-    (property "Reference" "IC4" (at 162.56 100.33 0)
+    (property "Reference" "IC2" (at 162.56 100.33 0)
       (effects (font (size 1.27 1.27)))
     )
@@
       (project "HSWR"
         (path "/51094070-255e-40e7-bed5-d199e288e5dd/00000000-0000-0000-0000-00005899e225"
-          (reference "IC4") (unit 1)
+          (reference "IC2") (unit 1)
         )
         (path "/51094070-255e-40e7-bed5-d199e288e5dd"
@@
   (symbol (lib_id "power:Earth") (at 144.78 68.58 0) (mirror y) (unit 1)
     (in_bom yes) (on_board yes) (dnp no)
-    (property "Reference" "#PWR0103" (at 144.78 74.93 0)
+    (property "Reference" "#PWR028" (at 144.78 74.93 0)
       (effects (font (size 1.27 1.27)) hide)
     )
@@
       (project "HSWR"
         (path "/51094070-255e-40e7-bed5-d199e288e5dd/00000000-0000-0000-0000-00005899e225"
-          (reference "#PWR0103") (unit 1)
+          (reference "#PWR028") (unit 1)
         )
       )
@@
   (symbol (lib_id "power:Earth") (at 110.49 71.12 0) (mirror y) (unit 1)
     (in_bom yes) (on_board yes) (dnp no)
-    (property "Reference" "#PWR0101" (at 110.49 77.47 0)
+    (property "Reference" "#PWR026" (at 110.49 77.47 0)
       (effects (font (size 1.27 1.27)) hide)
     )
@@
       (project "HSWR"
         (path "/51094070-255e-40e7-bed5-d199e288e5dd/00000000-0000-0000-0000-00005899e225"
-          (reference "#PWR0101") (unit 1)
+          (reference "#PWR026") (unit 1)
         )
       )
@@
   (symbol (lib_id "power:Earth") (at 146.05 102.87 0) (mirror y) (unit 1)
     (in_bom yes) (on_board yes) (dnp no)
-    (property "Reference" "#PWR0104" (at 146.05 109.22 0)
+    (property "Reference" "#PWR029" (at 146.05 109.22 0)
       (effects (font (size 1.27 1.27)) hide)
     )
@@
       (project "HSWR"
         (path "/51094070-255e-40e7-bed5-d199e288e5dd/00000000-0000-0000-0000-00005899e225"
-          (reference "#PWR0104") (unit 1)
+          (reference "#PWR029") (unit 1)
         )
       )
@@
   (symbol (lib_id "power:Earth") (at 148.59 102.87 0) (mirror y) (unit 1)
     (in_bom yes) (on_board yes) (dnp no)
-    (property "Reference" "#PWR0105" (at 148.59 109.22 0)
+    (property "Reference" "#PWR031" (at 148.59 109.22 0)
       (effects (font (size 1.27 1.27)) hide)
     )
@@
       (project "HSWR"
         (path "/51094070-255e-40e7-bed5-d199e288e5dd/00000000-0000-0000-0000-00005899e225"
-          (reference "#PWR0105") (unit 1)
+          (reference "#PWR031") (unit 1)
         )
       )
@@
   (symbol (lib_id "power:GND") (at 156.21 102.87 0) (unit 1)
     (in_bom yes) (on_board yes) (dnp no)
-    (property "Reference" "#PWR0107" (at 156.21 109.22 0)
+    (property "Reference" "#PWR033" (at 156.21 109.22 0)
       (effects (font (size 1.27 1.27)) hide)
     )
@@
       (project "HSWR"
         (path "/51094070-255e-40e7-bed5-d199e288e5dd/00000000-0000-0000-0000-00005899e225"
-          (reference "#PWR0107") (unit 1)
+          (reference "#PWR033") (unit 1)
         )
       )
@@
   (symbol (lib_id "power:GND") (at 158.75 102.87 0) (unit 1)
     (in_bom yes) (on_board yes) (dnp no)
-    (property "Reference" "#PWR0110" (at 158.75 109.22 0)
+    (property "Reference" "#PWR036" (at 158.75 109.22 0)
       (effects (font (size 1.27 1.27)) hide)
     )
@@
       (project "HSWR"
         (path "/51094070-255e-40e7-bed5-d199e288e5dd/00000000-0000-0000-0000-00005899e225"
-          (reference "#PWR0110") (unit 1)
+          (reference "#PWR036") (unit 1)
         )
       )
@@
   (symbol (lib_id "power:GND") (at 157.48 68.58 0) (unit 1)
     (in_bom yes) (on_board yes) (dnp no)
-    (property "Reference" "#PWR0109" (at 157.48 74.93 0)
+    (property "Reference" "#PWR035" (at 157.48 74.93 0)
       (effects (font (size 1.27 1.27)) hide)
     )
@@
       (project "HSWR"
         (path "/51094070-255e-40e7-bed5-d199e288e5dd/00000000-0000-0000-0000-00005899e225"
-          (reference "#PWR0109") (unit 1)
+          (reference "#PWR035") (unit 1)
         )
       )
@@
   (symbol (lib_id "power:+5VA") (at 148.59 63.5 0) (unit 1)
     (in_bom yes) (on_board yes) (dnp no)
-    (property "Reference" "#PWR0144" (at 148.59 67.31 0)
+    (property "Reference" "#PWR030" (at 148.59 67.31 0)
       (effects (font (size 1.27 1.27)) hide)
     )
@@
       (project "HSWR"
         (path "/51094070-255e-40e7-bed5-d199e288e5dd/00000000-0000-0000-0000-00005899e225"
-          (reference "#PWR0144") (unit 1)
+          (reference "#PWR030") (unit 1)
         )
       )
@@
   (symbol (lib_id "Regulator_Linear:AP1117-50") (at 118.11 63.5 0) (unit 1)
     (in_bom yes) (on_board yes) (dnp no)
-    (property "Reference" "U8" (at 118.11 57.3532 0)
+    (property "Reference" "U2" (at 118.11 57.3532 0)
       (effects (font (size 1.27 1.27)))
     )
@@
       (project "HSWR"
         (path "/51094070-255e-40e7-bed5-d199e288e5dd/00000000-0000-0000-0000-00005899e225"
-          (reference "U8") (unit 1)
-        )
-      )
+          (reference "U2") (unit 1)
+        )
+      )

Commit message: - some layout work
Parts:
- U2: symbol Regulator_Linear:AP1117-50 -> Regulator_Linear:L7805
Connections:
- net +12VA: now also U2.1 (IN); no longer U2.3 (VI)
- net +5VA: now also U2.3 (OUT); no longer U2.2 (VO)
- net Earth: now also U2.2 (GND); no longer U2.1 (GND)
Changed lines of the file:
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@@
       (effects (font (size 1.27 1.27)) hide)
     )
-    (property "Value" "+12VA" (at 110.871 59.1058 0)
+    (property "Value" "+12VA" (at 110.49 57.15 0)
       (effects (font (size 1.27 1.27)))
     )
@@
     )
   )
-  (symbol (lib_id "Regulator_Linear:AP1117-50") (at 118.11 63.5 0) (unit 1)
+  (symbol (lib_id "Regulator_Linear:L7805") (at 118.11 63.5 0) (unit 1)
     (in_bom yes) (on_board yes) (dnp no)
     (property "Reference" "U2" (at 118.11 57.3532 0)
@@
       (effects (font (size 1.27 1.27)))
     )
-    (property "Footprint" "Package_TO_SOT_SMD:SOT-223-3_TabPin2" (at 118.11 58.42 0)
-      (effects (font (size 1.27 1.27)) hide)
-    )
-    (property "Datasheet" "http://www.diodes.com/datasheets/AP1117.pdf" (at 120.65 69.85 0)
-      (effects (font (size 1.27 1.27)) hide)
-    )
+    (property "Footprint" "Package_TO_SOT_SMD:SOT-223-3_TabPin2" (at 118.745 67.31 0)
+      (effects (font (size 1.27 1.27) italic) (justify left) hide)
+    )
+    (property "Datasheet" "http://www.st.com/content/ccc/resource/technical/document/datasheet/41/4f/b3/b0/12/d4/47/88/CD00000444.pdf/files/CD00000444.pdf/jcr:content/translations/en.CD00000444.pdf" (at 118.11 64.77 0)
+      (effects (font (size 1.27 1.27)) hide)
+    )
