File: Supply.kicad_sch (KiCad schematic)
At the start: 14 parts, among them IC1 B1212S-2W, IC3 JW5052C

Commit message: - some work on schematic
Parts:
- renumbered C2 to C53, C4 to C54, C5 to C55, C6 to C56, C8 to C57, C9 to C58, C11 to C59, IC1 to IC3, IC3 to IC4, R13 to R47, R16 to R48, R17 to R49
