File: USB.kicad_sch (KiCad schematic)
At the start: 10 parts, among them IC5 ADuM4160

Commit message: - some work on schematic
Parts:
- renumbered C55 to C2, C56 to C3, C57 to C4, IC5 to IC1, R42 to R10, R43 to R11, R44 to R12, R45 to R13, R46 to R14, R41 to R9
Changed lines of the file:
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@@
   (symbol (lib_id "Interface_USB:ADUM4160") (at 144.78 95.25 0) (unit 1)
     (in_bom yes) (on_board yes) (dnp no)
-    (property "Reference" "IC5" (at 144.78 96.52 90)
+    (property "Reference" "IC1" (at 144.78 96.52 90)
       (effects (font (size 1.27 1.27)) (justify left))
     )
@@
       (project "HSWR"
         (path "/51094070-255e-40e7-bed5-d199e288e5dd/00000000-0000-0000-0000-00005ca14308"
-          (reference "IC5") (unit 1)
+          (reference "IC1") (unit 1)
         )
       )
@@
   (symbol (lib_id "Device:C") (at 130.81 106.68 0) (mirror x) (unit 1)
     (in_bom yes) (on_board yes) (dnp no)
-    (property "Reference" "C55" (at 127.889 105.5116 0)
+    (property "Reference" "C2" (at 127.889 105.5116 0)
       (effects (font (size 1.27 1.27)) (justify right))
     )
@@
       (project "HSWR"
         (path "/51094070-255e-40e7-bed5-d199e288e5dd/00000000-0000-0000-0000-00005ca14308"
-          (reference "C55") (unit 1)
+          (reference "C2") (unit 1)
         )
       )
@@
   (symbol (lib_id "Device:C") (at 138.43 72.39 0) (mirror x) (unit 1)
     (in_bom yes) (on_board yes) (dnp no)
-    (property "Reference" "C56" (at 135.509 71.2216 0)
+    (property "Reference" "C3" (at 135.509 71.2216 0)
       (effects (font (size 1.27 1.27)) (justify right))
     )
@@
       (project "HSWR"
         (path "/51094070-255e-40e7-bed5-d199e288e5dd/00000000-0000-0000-0000-00005ca14308"
-          (reference "C56") (unit 1)
+          (reference "C3") (unit 1)
         )
       )
@@
   (symbol (lib_id "Device:C") (at 158.75 106.68 180) (unit 1)
     (in_bom yes) (on_board yes) (dnp no)
-    (property "Reference" "C57" (at 161.671 105.5116 0)
+    (property "Reference" "C4" (at 161.671 105.5116 0)
       (effects (font (size 1.27 1.27)) (justify right))
     )
@@
       (project "HSWR"
         (path "/51094070-255e-40e7-bed5-d199e288e5dd/00000000-0000-0000-0000-00005ca14308"
-          (reference "C57") (unit 1)
+          (reference "C4") (unit 1)
         )
       )
@@
   (symbol (lib_id "power:GND") (at 158.75 110.49 0) (unit 1)
     (in_bom yes) (on_board yes) (dnp no)
-    (property "Reference" "#PWR0118" (at 158.75 116.84 0)
+    (property "Reference" "#PWR024" (at 158.75 116.84 0)
       (effects (font (size 1.27 1.27)) hide)
     )
@@
       (project "HSWR"
         (path "/51094070-255e-40e7-bed5-d199e288e5dd/00000000-0000-0000-0000-00005ca14308"
-          (reference "#PWR0118") (unit 1)
+          (reference "#PWR024") (unit 1)
         )
       )
@@
   (symbol (lib_id "power:+3V3") (at 147.32 67.31 0) (unit 1)
     (in_bom yes) (on_board yes) (dnp no)
-    (property "Reference" "#PWR0115" (at 147.32 71.12 0)
+    (property "Reference" "#PWR021" (at 147.32 71.12 0)
       (effects (font (size 1.27 1.27)) hide)
     )
@@
       (project "HSWR"
         (path "/51094070-255e-40e7-bed5-d199e288e5dd/00000000-0000-0000-0000-00005ca14308"
-          (reference "#PWR0115") (unit 1)
+          (reference "#PWR021") (unit 1)
         )
       )
@@
   (symbol (lib_id "power:GND") (at 149.86 110.49 0) (unit 1)
     (in_bom yes) (on_board yes) (dnp no)
-    (property "Reference" "#PWR0117" (at 149.86 116.84 0)
+    (property "Reference" "#PWR023" (at 149.86 116.84 0)
       (effects (font (size 1.27 1.27)) hide)
     )
@@
       (project "HSWR"
         (path "/51094070-255e-40e7-bed5-d199e288e5dd/00000000-0000-0000-0000-00005ca14308"
-          (reference "#PWR0117") (unit 1)
+          (reference "#PWR023") (unit 1)
         )
       )
@@
   (symbol (lib_id "power:GND") (at 147.32 110.49 0) (unit 1)
     (in_bom yes) (on_board yes) (dnp no)
-    (property "Reference" "#PWR0116" (at 147.32 116.84 0)
+    (property "Reference" "#PWR022" (at 147.32 116.84 0)
       (effects (font (size 1.27 1.27)) hide)
     )
@@
       (project "HSWR"
         (path "/51094070-255e-40e7-bed5-d199e288e5dd/00000000-0000-0000-0000-00005ca14308"
-          (reference "#PWR0116") (unit 1)
+          (reference "#PWR022") (unit 1)
         )
       )
@@
   (symbol (lib_id "Device:R") (at 114.3 95.25 270) (mirror x) (unit 1)
     (in_bom yes) (on_board yes) (dnp no)
-    (property "Reference" "R42" (at 114.3 97.79 90)
+    (property "Reference" "R10" (at 114.3 97.79 90)
       (effects (font (size 1.27 1.27)))
     )
@@
       (project "HSWR"
         (path "/51094070-255e-40e7-bed5-d199e288e5dd/00000000-0000-0000-0000-00005ca14308"
-          (reference "R42") (unit 1)
+          (reference "R10") (unit 1)
         )
       )
@@
   (symbol (lib_id "Device:R") (at 114.3 92.71 90) (mirror x) (unit 1)
     (in_bom yes) (on_board yes) (dnp no)
-    (property "Reference" "R41" (at 114.3 90.17 90)
+    (property "Reference" "R9" (at 114.3 90.17 90)
       (effects (font (size 1.27 1.27)))
     )
@@
       (project "HSWR"
         (path "/51094070-255e-40e7-bed5-d199e288e5dd/00000000-0000-0000-0000-00005ca14308"
-          (reference "R41") (unit 1)
+          (reference "R9") (unit 1)
         )
       )
@@
   (symbol (lib_id "Device:R") (at 175.26 95.25 270) (mirror x) (unit 1)
     (in_bom yes) (on_board yes) (dnp no)
-    (property "Reference" "R46" (at 175.26 97.79 90)
+    (property "Reference" "R14" (at 175.26 97.79 90)
       (effects (font (size 1.27 1.27)))
     )
@@
       (project "HSWR"
         (path "/51094070-255e-40e7-bed5-d199e288e5dd/00000000-0000-0000-0000-00005ca14308"
-          (reference "R46") (unit 1)
+          (reference "R14") (unit 1)
         )
       )
@@
   (symbol (lib_id "Device:R") (at 175.26 92.71 90) (mirror x) (unit 1)
     (in_bom yes) (on_board yes) (dnp no)
-    (property "Reference" "R45" (at 175.26 90.17 90)
+    (property "Reference" "R13" (at 175.26 90.17 90)
       (effects (font (size 1.27 1.27)))
     )
@@
       (project "HSWR"
         (path "/51094070-255e-40e7-bed5-d199e288e5dd/00000000-0000-0000-0000-00005ca14308"
-          (reference "R45") (unit 1)
+          (reference "R13") (unit 1)
         )
       )
@@
   (symbol (lib_id "power:GNDD") (at 142.24 110.49 0) (unit 1)
     (in_bom yes) (on_board yes) (dnp no)
-    (property "Reference" "#PWR0114" (at 142.24 116.84 0)
+    (property "Reference" "#PWR020" (at 142.24 116.84 0)
       (effects (font (size 1.27 1.27)) hide)
     )
@@
       (project "HSWR"
         (path "/51094070-255e-40e7-bed5-d199e288e5dd/00000000-0000-0000-0000-00005ca14308"
-          (reference "#PWR0114") (unit 1)
+          (reference "#PWR020") (unit 1)
         )
       )
@@
   (symbol (lib_id "power:GNDD") (at 139.7 110.49 0) (unit 1)
     (in_bom yes) (on_board yes) (dnp no)
-    (property "Reference" "#PWR0113" (at 139.7 116.84 0)
+    (property "Reference" "#PWR019" (at 139.7 116.84 0)
       (effects (font (size 1.27 1.27)) hide)
     )
@@
       (project "HSWR"
         (path "/51094070-255e-40e7-bed5-d199e288e5dd/00000000-0000-0000-0000-00005ca14308"
-          (reference "#PWR0113") (unit 1)
+          (reference "#PWR019") (unit 1)
         )
       )
@@
   (symbol (lib_id "power:GNDD") (at 130.81 110.49 0) (unit 1)
     (in_bom yes) (on_board yes) (dnp no)
-    (property "Reference" "#PWR0111" (at 130.81 116.84 0)
+    (property "Reference" "#PWR017" (at 130.81 116.84 0)
       (effects (font (size 1.27 1.27)) hide)
     )
@@
       (project "HSWR"
         (path "/51094070-255e-40e7-bed5-d199e288e5dd/00000000-0000-0000-0000-00005ca14308"
-          (reference "#PWR0111") (unit 1)
+          (reference "#PWR017") (unit 1)
         )
       )
@@
   (symbol (lib_id "power:GNDD") (at 138.43 76.2 0) (unit 1)
     (in_bom yes) (on_board yes) (dnp no)
-    (property "Reference" "#PWR0112" (at 138.43 82.55 0)
+    (property "Reference" "#PWR018" (at 138.43 82.55 0)
       (effects (font (size 1.27 1.27)) hide)
     )
@@
       (project "HSWR"
         (path "/51094070-255e-40e7-bed5-d199e288e5dd/00000000-0000-0000-0000-00005ca14308"
-          (reference "#PWR0112") (unit 1)
+          (reference "#PWR018") (unit 1)
         )
       )
@@
   (symbol (lib_id "Device:R") (at 144.78 125.73 270) (mirror x) (unit 1)
     (in_bom yes) (on_board yes) (dnp no)
-    (property "Reference" "R44" (at 144.78 128.27 90)
+    (property "Reference" "R12" (at 144.78 128.27 90)
       (effects (font (size 1.27 1.27)))
     )
@@
       (project "HSWR"
         (path "/51094070-255e-40e7-bed5-d199e288e5dd/00000000-0000-0000-0000-00005ca14308"
-          (reference "R44") (unit 1)
+          (reference "R12") (unit 1)
         )
       )
@@
   (symbol (lib_id "Device:R") (at 144.78 123.19 90) (mirror x) (unit 1)
     (in_bom yes) (on_board yes) (dnp no)
-    (property "Reference" "R43" (at 144.78 120.65 90)
+    (property "Reference" "R11" (at 144.78 120.65 90)
       (effects (font (size 1.27 1.27)))
     )
@@
       (project "HSWR"
         (path "/51094070-255e-40e7-bed5-d199e288e5dd/00000000-0000-0000-0000-00005ca14308"
-          (reference "R43") (unit 1)
-        )
-      )
+          (reference "R11") (unit 1)
+        )
+      )

Commit message: - layout almost finished
Parts:
- removed R11, R12: 0R, Resistor_SMD:R_0805_2012Metric, symbol Device:R
Other:
- note removed: "Optional if no isolation is required."
Changed lines of the file:
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@@
   (junction (at 158.75 87.63) (diameter 0) (color 0 0 0 0)
   )
-  (junction (at 170.18 92.71) (diameter 0) (color 0 0 0 0)
-  )
   (junction (at 158.75 85.09) (diameter 0) (color 0 0 0 0)
   )
   (junction (at 147.32 80.01) (diameter 0) (color 0 0 0 0)
   )
-  (junction (at 119.38 92.71) (diameter 0) (color 0 0 0 0)
-  )
   (junction (at 158.75 100.33) (diameter 0) (color 0 0 0 0)
   )
@@
   (junction (at 130.81 97.79) (diameter 0) (color 0 0 0 0)
   )
-  (junction (at 121.92 95.25) (diameter 0) (color 0 0 0 0)
-  )
-  (junction (at 167.64 95.25) (diameter 0) (color 0 0 0 0)
-  )
   (wire (pts (xy 158.75 100.33) (xy 158.75 102.87))
     (stroke (width 0) (type default))
   )
-  (wire (pts (xy 167.64 95.25) (xy 157.48 95.25))
-    (stroke (width 0) (type default))
-  )
-  (wire (pts (xy 121.92 95.25) (xy 132.08 95.25))
-    (stroke (width 0) (type default))
-  )
-  (wire (pts (xy 170.18 125.73) (xy 170.18 92.71))
-    (stroke (width 0) (type default))
-  )
-  (wire (pts (xy 119.38 92.71) (xy 118.11 92.71))
+  (wire (pts (xy 157.48 95.25) (xy 171.45 95.25))
+    (stroke (width 0) (type default))
+  )
+  (wire (pts (xy 118.11 92.71) (xy 132.08 92.71))
     (stroke (width 0) (type default))
   )
@@
     (stroke (width 0) (type default))
   )
-  (wire (pts (xy 140.97 123.19) (xy 121.92 123.19))
-    (stroke (width 0) (type default))
-  )
   (wire (pts (xy 147.32 80.01) (xy 158.75 80.01))
     (stroke (width 0) (type default))
   )
-  (wire (pts (xy 171.45 92.71) (xy 170.18 92.71))
-    (stroke (width 0) (type default))
-  )
   (wire (pts (xy 130.81 85.09) (xy 132.08 85.09))
     (stroke (width 0) (type default))
   )
-  (wire (pts (xy 171.45 95.25) (xy 167.64 95.25))
-    (stroke (width 0) (type default))
-  )
   (wire (pts (xy 130.81 100.33) (xy 130.81 102.87))
     (stroke (width 0) (type default))
   )
-  (wire (pts (xy 148.59 123.19) (xy 167.64 123.19))
-    (stroke (width 0) (type default))
-  )
-  (wire (pts (xy 119.38 92.71) (xy 119.38 125.73))
-    (stroke (width 0) (type default))
-  )
-  (wire (pts (xy 132.08 92.71) (xy 119.38 92.71))
-    (stroke (width 0) (type default))
-  )
   (wire (pts (xy 147.32 67.31) (xy 147.32 80.01))
     (stroke (width 0) (type default))
   )
-  (wire (pts (xy 170.18 92.71) (xy 157.48 92.71))
+  (wire (pts (xy 157.48 92.71) (xy 171.45 92.71))
     (stroke (width 0) (type default))
   )
@@
     (stroke (width 0) (type default))
   )
-  (wire (pts (xy 118.11 95.25) (xy 121.92 95.25))
-    (stroke (width 0) (type default))
-  )
-  (wire (pts (xy 148.59 125.73) (xy 170.18 125.73))
-    (stroke (width 0) (type default))
-  )
-  (wire (pts (xy 121.92 123.19) (xy 121.92 95.25))
+  (wire (pts (xy 118.11 95.25) (xy 132.08 95.25))
     (stroke (width 0) (type default))
   )
@@
   (wire (pts (xy 157.48 100.33) (xy 158.75 100.33))
     (stroke (width 0) (type default))
-  )
-  (wire (pts (xy 167.64 123.19) (xy 167.64 95.25))
-    (stroke (width 0) (type default))
-  )
-  (wire (pts (xy 119.38 125.73) (xy 140.97 125.73))
-    (stroke (width 0) (type default))
-  )
-  (text "Optional if no isolation is required." (at 128.27 132.08 0)
-    (effects (font (size 1.27 1.27)) (justify left bottom))
   )
   (hierarchical_label "Host_D-" (shape bidirectional) (at 110.49 95.25 180) (fields_autoplaced)
@@
         )
       )
-    )
-  )
-  (symbol (lib_id "Device:R") (at 144.78 125.73 270) (mirror x) (unit 1)
-    (in_bom yes) (on_board yes) (dnp no)
-    (property "Reference" "R12" (at 144.78 128.27 90)
-      (effects (font (size 1.27 1.27)))
-    )
-    (property "Value" "0R" (at 144.78 125.73 90)
-      (effects (font (size 1.27 1.27)))
-    )
-    (property "Footprint" "Resistor_SMD:R_0805_2012Metric" (at 144.78 127.508 90)
-      (effects (font (size 1.27 1.27)) hide)
-    )
-    (property "Datasheet" "~" (at 144.78 125.73 0)
-      (effects (font (size 1.27 1.27)) hide)
-    )
-    (pin "1")
-    (pin "2")
-    (instances
-      (project "HSWR"
-        (path "/51094070-255e-40e7-bed5-d199e288e5dd/00000000-0000-0000-0000-00005ca14308"
-          (reference "R12") (unit 1)
-        )
-      )
-    )
-  )
-  (symbol (lib_id "Device:R") (at 144.78 123.19 90) (mirror x) (unit 1)
-    (in_bom yes) (on_board yes) (dnp no)
-    (property "Reference" "R11" (at 144.78 120.65 90)
-      (effects (font (size 1.27 1.27)))
-    )
-    (property "Value" "0R" (at 144.78 123.19 90)
-      (effects (font (size 1.27 1.27)))
-    )
-    (property "Footprint" "Resistor_SMD:R_0805_2012Metric" (at 144.78 121.412 90)
-      (effects (font (size 1.27 1.27)) hide)
-    )
-    (property "Datasheet" "~" (at 144.78 123.19 0)
-      (effects (font (size 1.27 1.27)) hide)
-    )
-    (pin "1")
-    (pin "2")
-    (instances
-      (project "HSWR"
-        (path "/51094070-255e-40e7-bed5-d199e288e5dd/00000000-0000-0000-0000-00005ca14308"
-          (reference "R11") (unit 1)
-        )
-      )
