File: iso_IO.kicad_sch (KiCad schematic)
At the start: 32 parts, among them J9 AVR-ISP-6, Q7 Q_NMOS_GDS, U10 AM26LV32xD, U11 ADuM120N1, U12 ADuM120N1, U13 PC355, U9 ATtiny13A-SU

Commit message: - some work on schematic
Parts:
- removed C49, C59: 100n, Capacitor_SMD:C_0805_2012Metric, symbol Device:C
- removed JP1: H1, Jumper:SolderJumper-2_P1.3mm_Open_TrianglePad1.0x1.5mm, symbol Jumper:Jumper_2_Open
- removed JP3: H2, Jumper:SolderJumper-2_P1.3mm_Open_TrianglePad1.0x1.5mm, symbol Jumper:Jumper_2_Open
- removed JP4: H3, Jumper:SolderJumper-2_P1.3mm_Open_TrianglePad1.0x1.5mm, symbol Jumper:Jumper_2_Open
- removed JP5: EN, Jumper:SolderJumper-3_P2.0mm_Open_TrianglePad1.0x1.5mm, symbol HSWR-rescue:SolderJumper_3_Open-Jumper
- removed R3, R33, R34, R4: 120R, Resistor_SMD:R_0805_2012Metric, symbol Device:R_Small
- removed R37: 100R, Resistor_SMD:R_0805_2012Metric, symbol Device:R
- removed U10: AM26LV32xD, Package_SO:SOIC-16_3.9x9.9mm_P1.27mm, symbol Interface:AM26LV32xD
- removed U11, U12: ADuM120N1, Package_SO:SOIC-8_3.9x4.9mm_P1.27mm, symbol Isolator:ADuM120N
- removed U13: PC355, Package_SO:SO-4_4.4x4.3mm_P2.54mm, symbol Isolator:SFH617A-1
- added C10: 100n, Capacitor_SMD:C_0805_2012Metric, symbol Device:C
- added U5: ADuM120N, Package_SO:SOIC-8_3.9x4.9mm_P1.27mm, symbol Isolator:ADuM120N
- added U6: ADuM261N, Package_SO:SOIC-16W_7.5x12.8mm_P1.27mm, symbol Isolator:ADuM261N
- renumbered C60 to C11, C50 to C12, C51 to C13, C58 to C14, C62 to C8, C48 to C9, J9 to J11, Q7 to Q1, R1 to R16, R2 to R17, R35 to R22, R38 to R23, R39 to R24, R47 to R25, R48 to R26, R36 to R27, U9 to U3
Connections:
- net +3V3: now also C10.1, U5.8 (VDD2), U6.16 (VDD2)
- net +5VA: now also U6.1 (VDD1)
- net Earth: now also U6.8 (GND1)
- net GND: now also C10.2, U5.5 (GND2), U6.9 (GND2)
- net UART: now also U5.6 (VOB)
- new net Fan: U6.10 (VIF)
- new net H1_A: U6.15 (VOA)
- new net H1_B: U6.14 (VOB)
- new net H1_C: U6.13 (VOC)
- new net H2_A: U6.12 (VOD)
- new net H2_B: U6.11 (VOE)
- new net H2_C: U5.7 (VOA)
- no-connect marks 1 -> 0
Other:
- moved on the sheet: C12, C14

Commit message: - some layout work
Parts:
- removed R23, R24, R25: 10k, Resistor_SMD:R_0805_2012Metric, symbol Device:R
- added R18: 100R, Resistor_SMD:R_0805_2012Metric, symbol Device:R
- added R19: 1k, Resistor_SMD:R_0805_2012Metric, symbol Device:R
- added R20: 10k, Resistor_SMD:R_0805_2012Metric, symbol Device:R
- added RN1, RN2: 10k, Resistor_SMD:R_Array_Convex_4x0603, symbol Device:R_Pack04
- C13: value 100n -> 10n
- U3: footprint Package_SO:SOIJ-8_5.3x5.3mm_P1.27mm -> Package_SO:SO-8_5.3x6.2mm_P1.27mm
Connections:
- net +5VA: now also U5.1 (VDD1), R20.1, RN1.6 (R3.2), RN1.7 (R2.2), RN1.8 (R1.2), RN2.2 (R2.1), RN2.3 (R3.1), RN2.4 (R4.1); no longer C13.1
- net Earth: now also U5.4 (GND1)
- net Hall1_A: now also U6.2 (VIA), RN1.1 (R1.1)
- net Hall1_B: now also U6.3 (VIB), RN1.2 (R2.1)
- net Hall1_C: now also U6.4 (VIC), RN1.3 (R3.1)
- net at Q1.1 (G), R27.1: now also U6.7 (VOF)
- net at R17.1, U3.2 (PB3): now also R19.1
- net at J11.4 (MOSI), R16.1, U3.5 (PB0): now also R18.1
- net M2_Temp: now reaches J11.1 (MISO), U3.6 (PB1)
- net M2_Temp: now also C13.1, R18.2, R19.2, R20.2
- net at J11.3 (SCK), U3.7 (PB2): now also U5.3 (VIB)
- net Hall2_A: now reaches U6.5 (VID)
- net Hall2_A: now also RN2.7 (R2.2)
- net Hall2_B: now reaches U6.6 (VIE)
- net Hall2_B: now also RN2.6 (R3.2)
- net Hall2_C: now reaches U5.2 (VIA)
- net Hall2_C: now also RN2.5 (R4.2)
- net M_Temp renamed M1_Temp
- no-connect marks 0 -> 4
Other:
- moved on the sheet: C12, C8, Q1, R16, R17, R22, R26, R27
